File: hardware/kicad/01B_ACC_WAKE.kicad_sch (KiCad schematic)
At the start: 9 parts, among them Q301 MMBT5551 (C408396), Q302 MMBT5401 (C408397)

Commit message: hardware(kicad): add 01C TLC555-Q1 max relay hold timer and gated MCU hold signal
Parts:
- added R305: 100k ACC_DRIVE_OFF_PULLDOWN, Tripmaster:R_1206_3216, symbol Tripmaster_Sym:R
Connections:
- net ACC_DRIVE_5V: now also R305.1
- net GND: now also R305.2
Changed lines of the file:
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@@
 (text "HOLD TIMER and BAT_SW vehicle-only interlock NOT DESIGNED: USB-only must NEVER energize K101." (at 196 261 0) (effects (font (size 1.16 1.16))))
 (text "No ERC/DRC. 30V Schottky diodes used ONLY on <=5V logic paths, NOT raw vehicle ACC." (at 196 272 0) (effects (font (size 1.18 1.18))))
- (sheet_instances (path "/a26d9b0c-7f10-4e5a-a65f-000000000064/a26d9b0c-7f10-4e5a-a65f-000000000065" (page "2.2")))
+ (symbol (lib_id "Tripmaster_Sym:R") (at 380 190 0) (unit 1) (exclude_from_sim no) (in_bom yes) (on_board yes) (dnp no)
+(property "Reference" "R305" (at 380 172 0) (effects (font (size 1.27 1.27))))
+(property "Value" "100k ACC_DRIVE_OFF_PULLDOWN" (at 380 175 0) (effects (font (size 1.27 1.27))))
+(property "Footprint" "Tripmaster:R_1206_3216" (at 380 190 0) (effects (font (size 1.27 1.27)) (hide yes)))
+(pin "1")
+(pin "2")
+(instances (project "TripTracer_V1" (path "/a26d9b0c-7f10-4e5a-a65f-000000000064/a26d9b0c-7f10-4e5a-a65f-000000000065/be2301bb-8455-4581-8a01-3333333301bb" (reference "R305") (unit 1)))))
+(wire (pts (xy 368.57 190) (xy 358 190)) (stroke (width 0) (type default)))
+(global_label "ACC_DRIVE_5V" (shape bidirectional) (at 358 190 0) (effects (font (size 1.27 1.27)) (justify left)))
+(wire (pts (xy 391.43 190) (xy 403 190)) (stroke (width 0) (type default)))
+(global_label "GND" (shape bidirectional) (at 403 190 0) (effects (font (size 1.27 1.27)) (justify left)))
+(sheet_instances (path "/a26d9b0c-7f10-4e5a-a65f-000000000064/a26d9b0c-7f10-4e5a-a65f-000000000065" (page "2.2")))
  (embedded_fonts no)
 )
