File: hardware/kicad/01F_RC_SHUTDOWN.kicad_sch (KiCad schematic)
At the start: 7 parts, among them Q801 DMN2056U discharge only

Commit message: hardware(kicad): align RC discharge MOSFET pins and wires on 1.27 mm grid
Parts:
- Q801: symbol Tripmaster_Sym:NMOS -> TripTracer_V1:NMOS_GDS_127
Changed lines of the file:
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@@
 (wire (pts (xy 189.23 127) (xy 208.28 127)) (stroke (width 0) (type default)))
 (global_label "GND" (shape bidirectional) (at 208.28 127 0) (effects (font (size 1.27 1.27)) (justify left)))
-(symbol (lib_id "Tripmaster_Sym:NMOS") (at 217.17 176.53 0) (unit 1) (exclude_from_sim no) (in_bom yes) (on_board yes) (dnp no) (property "Reference" "Q801" (at 217.17 156.21 0) (effects (font (size 1.27 1.27)))) (property "Value" "DMN2056U discharge only" (at 217.17 160.02 0) (effects (font (size 1.27 1.27)))) (property "Footprint" "Tripmaster:Q1_Diodes_DMN2056U_7" (at 217.17 176.53 0) (effects (font (size 1.27 1.27)) (hide yes))) (pin "1")
+(symbol (lib_id "TripTracer_V1:NMOS_GDS_127") (at 217.17 176.53 0) (unit 1) (exclude_from_sim no) (in_bom yes) (on_board yes) (dnp no) (property "Reference" "Q801" (at 217.17 156.21 0) (effects (font (size 1.27 1.27)))) (property "Value" "DMN2056U discharge only" (at 217.17 160.02 0) (effects (font (size 1.27 1.27)))) (property "Footprint" "Tripmaster:Q1_Diodes_DMN2056U_7" (at 217.17 176.53 0) (effects (font (size 1.27 1.27)) (hide yes))) (pin "1")
 (pin "2")
 (pin "3") (instances (project "TripTracer_V1" (path "/a26d9b0c-7f10-4e5a-a65f-000000000064/a26d9b0c-7f10-4e5a-a65f-000000000065/10ca8836-c895-420f-ae42-aeb901d0b1a0" (reference "Q801") (unit 1)))))
-(wire (pts (xy 202.09 176.53) (xy 186.85 176.53)) (stroke (width 0) (type default)))
-(global_label "DISCHARGE_GATE" (shape bidirectional) (at 186.85 176.53 0) (effects (font (size 1.27 1.27)) (justify left)))
-(wire (pts (xy 232.25 173.99) (xy 252.57 173.99)) (stroke (width 0) (type default)))
-(global_label "HOLD_CAP_5V" (shape bidirectional) (at 252.57 173.99 0) (effects (font (size 1.27 1.27)) (justify left)))
-(wire (pts (xy 232.25 179.07) (xy 252.57 179.07)) (stroke (width 0) (type default)))
-(global_label "GND" (shape bidirectional) (at 252.57 179.07 0) (effects (font (size 1.27 1.27)) (justify left)))
+(wire (pts (xy 201.93 176.53) (xy 186.69 176.53)) (stroke (width 0) (type default)))
+(global_label "DISCHARGE_GATE" (shape bidirectional) (at 186.69 176.53 0) (effects (font (size 1.27 1.27)) (justify left)))
+(wire (pts (xy 232.41 173.99) (xy 252.73 173.99)) (stroke (width 0) (type default)))
+(global_label "HOLD_CAP_5V" (shape bidirectional) (at 252.73 173.99 0) (effects (font (size 1.27 1.27)) (justify left)))
+(wire (pts (xy 232.41 179.07) (xy 252.73 179.07)) (stroke (width 0) (type default)))
+(global_label "GND" (shape bidirectional) (at 252.73 179.07 0) (effects (font (size 1.27 1.27)) (justify left)))
 (symbol (lib_id "Tripmaster_Sym:R") (at 123.19 176.53 0) (unit 1) (exclude_from_sim no) (in_bom yes) (on_board yes) (dnp no) (property "Reference" "R803" (at 123.19 156.21 0) (effects (font (size 1.27 1.27)))) (property "Value" "10k MCU gate series" (at 123.19 160.02 0) (effects (font (size 1.27 1.27)))) (property "Footprint" "Tripmaster:R_1206_3216" (at 123.19 176.53 0) (effects (font (size 1.27 1.27)) (hide yes))) (pin "1")
 (pin "2") (instances (project "TripTracer_V1" (path "/a26d9b0c-7f10-4e5a-a65f-000000000064/a26d9b0c-7f10-4e5a-a65f-000000000065/10ca8836-c895-420f-ae42-aeb901d0b1a0" (reference "R803") (unit 1)))))

Commit message: fix(kicad): correct D801 NC pin and clean unused connection in 01F
Connections:
- net RC_CHG_LIMITED: no longer D801.2 (A2)
Changed lines of the file:
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@@
 (wire (pts (xy 83.82 96.52) (xy 71.12 96.52)) (stroke (width 0) (type default)))
 (global_label "RC_CHG_LIMITED" (shape bidirectional) (at 71.12 96.52 0) (effects (font (size 1.27 1.27)) (justify left)))
-(wire (pts (xy 83.82 106.68) (xy 71.12 106.68)) (stroke (width 0) (type default)))
-(global_label "RC_CHG_LIMITED" (shape bidirectional) (at 71.12 106.68 0) (effects (font (size 1.27 1.27)) (justify left)))
 (wire (pts (xy 129.54 101.6) (xy 148.59 101.6)) (stroke (width 0) (type default)))
 (global_label "HOLD_CAP_5V" (shape bidirectional) (at 148.59 101.6 0) (effects (font (size 1.27 1.27)) (justify left)))
