File: hardware/kicad/01D_INPUT_PROTECTION.kicad_sch (KiCad schematic)
At the start: 9 parts, among them Q401 IPD90N10S4-06 PROVISIONAL 100V, Q402 IPD90N10S4-06 PROVISIONAL 100V, U401 LM74930QRGERQ1_INCOMPLETE

Commit message: hardware(power): move surge-exposed Q401 candidate to 250V AEC-Q101 Infineon D2PAK
Parts:
- Q401: value IPD90N10S4-06 PROVISIONAL 100V -> IPB17N25S3-100 PROVISIONAL 250V; footprint Package_TO_SOT_SMD:TO-252-3_TabPin2 -> Package_TO_SOT_SMD:TO-263-3_TabPin2; symbol TripTracer_V1:IPD90N10S4_06 -> TripTracer_V1:IPB17N25S3_100

Commit message: cost(power): switch Q401 to lower-cost onsemi FQD16N25CTM, preserve pinout and provisional safety status
Parts:
- Q401: value IPB17N25S3-100 PROVISIONAL 250V -> FQD16N25CTM LOW-COST 250V PROVISIONAL; footprint Package_TO_SOT_SMD:TO-263-3_TabPin2 -> Package_TO_SOT_SMD:TO-252-3_TabPin2; symbol TripTracer_V1:IPB17N25S3_100 -> TripTracer_V1:FQD16N25CTM
