File: hardware/kicad/01C_HOLD_TIMER.kicad_sch (KiCad schematic)
At the start: 13 parts, among them U501 TLC555QDRQ1 - MONOSTABLE 24s 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, U502 SN74LVC1G08-Q1 AND

Commit message: hardware(power): use actual powered V3V3_SYS consistently for 555 timer and core
Connections:
- net 3V3_MAIN renamed V3V3_SYS
Changed lines of the file:
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@@
 (instances (project "TripTracer_V1" (path "/a26d9b0c-7f10-4e5a-a65f-000000000064/a26d9b0c-7f10-4e5a-a65f-000000000065/44e29570-df14-4b18-a1c0-222222222201" (reference "U502") (unit 1)))))
 (wire (pts (xy 147.14 94.76) (xy 119 94.76)) (stroke (width 0) (type default)))
-(global_label "3V3_MAIN" (shape bidirectional) (at 119 94.76 0) (effects (font (size 1.27 1.27)) (justify left)))
+(global_label "V3V3_SYS" (shape bidirectional) (at 119 94.76 0) (effects (font (size 1.27 1.27)) (justify left)))
 (wire (pts (xy 147.14 99.84) (xy 119 99.84)) (stroke (width 0) (type default)))
 (global_label "TIMER_TRIG" (shape bidirectional) (at 119 99.84 0) (effects (font (size 1.27 1.27)) (justify left)))
@@
 (global_label "HOLD_TIMER_GRANTED_3V3" (shape bidirectional) (at 351 110 0) (effects (font (size 1.27 1.27)) (justify left)))
 (wire (pts (xy 310 94.76) (xy 310 84)) (stroke (width 0) (type default)))
-(global_label "3V3_MAIN" (shape bidirectional) (at 310 84 0) (effects (font (size 1.27 1.27)) (justify left)))
+(global_label "V3V3_SYS" (shape bidirectional) (at 310 84 0) (effects (font (size 1.27 1.27)) (justify left)))
 (wire (pts (xy 310 125.24) (xy 310 138)) (stroke (width 0) (type default)))
 (global_label "GND" (shape bidirectional) (at 310 138 0) (effects (font (size 1.27 1.27)) (justify left)))
@@
 (instances (project "TripTracer_V1" (path "/a26d9b0c-7f10-4e5a-a65f-000000000064/a26d9b0c-7f10-4e5a-a65f-000000000065/44e29570-df14-4b18-a1c0-222222222201" (reference "R501") (unit 1)))))
 (wire (pts (xy 223.57 162) (xy 215 162)) (stroke (width 0) (type default)))
-(global_label "3V3_MAIN" (shape bidirectional) (at 215 162 0) (effects (font (size 1.27 1.27)) (justify left)))
+(global_label "V3V3_SYS" (shape bidirectional) (at 215 162 0) (effects (font (size 1.27 1.27)) (justify left)))
 (wire (pts (xy 246.43 162) (xy 255 162)) (stroke (width 0) (type default)))
 (global_label "TIMER_RC" (shape bidirectional) (at 255 162 0) (effects (font (size 1.27 1.27)) (justify left)))
@@
 (instances (project "TripTracer_V1" (path "/a26d9b0c-7f10-4e5a-a65f-000000000064/a26d9b0c-7f10-4e5a-a65f-000000000065/44e29570-df14-4b18-a1c0-222222222201" (reference "R502") (unit 1)))))
 (wire (pts (xy 58.57 169) (xy 50 169)) (stroke (width 0) (type default)))
-(global_label "3V3_MAIN" (shape bidirectional) (at 50 169 0) (effects (font (size 1.27 1.27)) (justify left)))
+(global_label "V3V3_SYS" (shape bidirectional) (at 50 169 0) (effects (font (size 1.27 1.27)) (justify left)))
 (wire (pts (xy 81.43 169) (xy 90 169)) (stroke (width 0) (type default)))
 (global_label "TIMER_TRIG" (shape bidirectional) (at 90 169 0) (effects (font (size 1.27 1.27)) (justify left)))
@@
 (instances (project "TripTracer_V1" (path "/a26d9b0c-7f10-4e5a-a65f-000000000064/a26d9b0c-7f10-4e5a-a65f-000000000065/44e29570-df14-4b18-a1c0-222222222201" (reference "R503") (unit 1)))))
 (wire (pts (xy 108.57 164) (xy 100 164)) (stroke (width 0) (type default)))
-(global_label "3V3_MAIN" (shape bidirectional) (at 100 164 0) (effects (font (size 1.27 1.27)) (justify left)))
+(global_label "V3V3_SYS" (shape bidirectional) (at 100 164 0) (effects (font (size 1.27 1.27)) (justify left)))
 (wire (pts (xy 131.43 164) (xy 140 164)) (stroke (width 0) (type default)))
 (global_label "TIMER_RESET" (shape bidirectional) (at 140 164 0) (effects (font (size 1.27 1.27)) (justify left)))
@@
 (instances (project "TripTracer_V1" (path "/a26d9b0c-7f10-4e5a-a65f-000000000064/a26d9b0c-7f10-4e5a-a65f-000000000065/44e29570-df14-4b18-a1c0-222222222201" (reference "C505") (unit 1)))))
 (wire (pts (xy 203.57 240) (xy 195 240)) (stroke (width 0) (type default)))
-(global_label "3V3_MAIN" (shape bidirectional) (at 195 240 0) (effects (font (size 1.27 1.27)) (justify left)))
+(global_label "V3V3_SYS" (shape bidirectional) (at 195 240 0) (effects (font (size 1.27 1.27)) (justify left)))
 (wire (pts (xy 226.43 240) (xy 235 240)) (stroke (width 0) (type default)))
 (global_label "GND" (shape bidirectional) (at 235 240 0) (effects (font (size 1.27 1.27)) (justify left)))
@@
 (global_label "TIMER_TRIG" (shape bidirectional) (at 44 256 0) (effects (font (size 1.27 1.27)) (justify left)))
 (wire (pts (xy 81.43 256) (xy 95 256)) (stroke (width 0) (type default)))
-(global_label "3V3_MAIN" (shape bidirectional) (at 95 256 0) (effects (font (size 1.27 1.27)) (justify left)))
+(global_label "V3V3_SYS" (shape bidirectional) (at 95 256 0) (effects (font (size 1.27 1.27)) (justify left)))
 (symbol (lib_id "Tripmaster_Sym:SCHOTTKY") (at 150 256 0) (unit 1) (exclude_from_sim no) (in_bom yes) (on_board yes) (dnp no)
 (property "Reference" "D502" (at 150 237 0) (effects (font (size 1.27 1.27))))
