File: hardware/kicad/01H_ACC_HOLD_GATE.kicad_sch (KiCad schematic)
At the start: 10 parts, among them U911 EL817S HOLD OPTICAL, U912 EL817S ACC SENSE

Commit message: fix(power): feed ACC optoisolator collector from real V3V3_SYS rail
Connections:
- net 3V3_MAIN renamed V3V3_SYS

Commit message: safety(power): replace obsolete 35V EL817S with 80V Wuerth 140356145000 optocouplers
Parts:
- R914: value 470R HOLD LED -> 330R HOLD LED
- R917: value 10k ACC SENSE BLEED -> 47k ACC SENSE BLEED
- U911: value EL817S HOLD OPTICAL -> 140356145000 HOLD OPTICAL; footprint Package_DIP:SMDIP-4_W7.62mm -> Tripmaster:Wurth_140356145000_SOP4; symbol TripTracer_V1:EL817S -> TripTracer_V1:WE_140356145000
- U912: value EL817S ACC SENSE -> 140356145000 ACC SENSE; footprint Package_DIP:SMDIP-4_W7.62mm -> Tripmaster:Wurth_140356145000_SOP4; symbol TripTracer_V1:EL817S -> TripTracer_V1:WE_140356145000

Commit message: hardware(acc): replace unqualified low-IF ACC optocoupler with two 160V-rated MMBT5551 inverters
Parts:
- removed U912: 140356145000 ACC SENSE, Tripmaster:Wurth_140356145000_SOP4, symbol TripTracer_V1:WE_140356145000
- added Q912, Q913: MMBT5551, Tripmaster:Q_SOT23_1B2E3C, symbol TripTracer_V1:MMBT5551
- added R918: 100k base leak pull-down, Tripmaster:R_1206_3216, symbol Tripmaster_Sym:R
- added R919: 22k first collector pull-up, Tripmaster:R_1206_3216, symbol Tripmaster_Sym:R
- added R920: 22k second base feed, Tripmaster:R_1206_3216, symbol Tripmaster_Sym:R
- added R921: 10k ACC output pull-up, Tripmaster:R_1206_3216, symbol Tripmaster_Sym:R
- R916: value 6.8k ACC LED -> 100k ACC NPN base feed
- R917: value 47k ACC SENSE BLEED -> 47k ACC output pulldown
Connections:
- net ACC_DRIVE_5V: now also Q913.3 (C), R921.2
- net GND: now also Q912.2 (E), Q913.2 (E), R918.2
- net V3V3_SYS: now also R919.1, R921.1
- net ACC_LED_ANODE renamed ACC_Q912_BASE
- net ACC_Q912_BASE: now also Q912.1 (B), R918.1
- new net ACC_INV_N: Q912.3 (C), R919.2, R920.1
- new net ACC_Q913_BASE: Q913.1 (B), R920.2
Other:
- note added: "CRITICAL: photocoupler U911 VCEO, CTR at -40C and LED current; Q912/Q913 BJT beta, VBE at hot/cold, ACC base resistor leakage, exact pinout/footprint, 9V and 30V thresholds, ACC transient protection, 01C 555 proper trigger and 3V3 power, power-on behavior ALL REQUIRE VERIFICATION. DO NOT FABRICATE."
- note added: "PROTOTYPE: ACC resistor divider + D911 BAT54 (A=1, K=2) starts EN independent of 5V. Opto U911 powered by VIN permits post-ACC MCU_HOLD only during independent 555 grant. Q912/Q913 double NPN stage generates non-inverted 3V3 ACC sense for the existing 555 falling-edge trigger; no CTR assumption."
- note removed: "CRITICAL: photocoupler U911 VCEO, CTR at -40C and LED current, exact pinout/footprint, 9V and 30V thresholds, ACC transient protection, 01C 555 proper trigger and 3V3 power, power-on behavior ALL REQUIRE VERIFICATION. DO NOT FABRICATE."
- note removed: "PROTOTYPE: ACC resistor divider + D911 BAT54 (A=1, K=2) starts EN independent of 5V. Opto U911 powered by VIN permits post-ACC MCU_HOLD only during independent 555 grant. U912 optically generates 3V3-level ACC sense for 01C trigger."
