File: hardware/kicad/04_ESP32_USB.kicad_sch (KiCad schematic)
At the start: 0 parts

Commit message: hardware: wire ESP32-S3 and native USB-C with CC pulls and ESD in V1
Parts:
- added C201: 100nF MCU local, Tripmaster:C_1210_3225, symbol Tripmaster_Sym:C1210
- added C202: 22uF MCU bulk, Tripmaster:C_1210_3225, symbol Tripmaster_Sym:C1210
- added C203: 1uF EN RC, Tripmaster:C_1210_3225, symbol Tripmaster_Sym:C1210
- added D201: USBLC6-2SC6, Tripmaster:D2_ST_USBLC6_2SC6, symbol Tripmaster_Sym:USB_ESD
- added J201: GCT USB4105-GF-A, Tripmaster:J1_GCT_USB4105_GF_A_USB_C, symbol Tripmaster_Sym:USB_C_GCT_USB4105
- added R201: 5.1k CC1, Tripmaster:R_1206_3216, symbol Tripmaster_Sym:R
- added R202: 5.1k CC2, Tripmaster:R_1206_3216, symbol Tripmaster_Sym:R
- added R203: 22R D+, Tripmaster:R_1206_3216, symbol Tripmaster_Sym:R
- added R204: 22R D-, Tripmaster:R_1206_3216, symbol Tripmaster_Sym:R
- added R205: 10k BOOT PU, Tripmaster:R_1206_3216, symbol Tripmaster_Sym:R
- added R206: 10k EN PU, Tripmaster:R_1206_3216, symbol Tripmaster_Sym:R
- added U201: ESP32-S3-MINI-1-N8, Tripmaster:U1_ESP32-S3-MINI-1-N8, symbol Tripmaster_Sym:ESP32_S3_MINI_1_N8
Connections:
- new net: J201.A5 (CC1), R201.2
- new net: J201.B5 (CC2), R202.1
- new net: D201.6 (IO1_OUT), R203.1
- new net BOOT0_RECOVERY: R205.1, U201.4 (IO0)
- new net EN_RESET: C203.2, R206.1, U201.45 (EN)
- new net GND: C201.1, C202.1, C203.1, D201.2 (GND), J201.A1 (GND_A1), J201.A12 (GND_A12), J201.B1 (GND_B1), J201.B12 (GND_B12), J201.SH (SHIELD), R201.1, R202.2, U201.1 (GND), U201.2 (GND), U201.42 (GND), U201.43 (GND), U201.46 (GND), U201.47 (GND), U201.48 (GND), U201.49 (GND), U201.50 (GND), U201.51 (GND), U201.52 (GND), U201.53 (GND), U201.54 (GND), U201.55 (GND), U201.56 (GND), U201.57 (GND), U201.58 (GND), U201.59 (GND), U201.60 (GND), U201.61 (GND), U201.62 (GND), U201.63 (GND), U201.64 (GND), U201.65 (GND)
- new net USB_DM_MCU: R204.2, U201.23 (IO19_USB_DM)
- new net USB_DM_PORT: D201.3 (IO2_IN), J201.A7 (D-_A7), J201.B7 (D-_B7)
- new net USB_DM_PORT_ESD: D201.4 (IO2_OUT), R204.1
- new net USB_DP_MCU: R203.2, U201.24 (IO20_USB_DP)
- new net USB_DP_PORT: D201.1 (IO1_IN), J201.A6 (D+_A6), J201.B6 (D+_B6)
- new net USB_VBUS_RAW: D201.5 (VBUS), J201.A4 (VBUS_A4), J201.A9 (VBUS_A9), J201.B4 (VBUS_B4), J201.B9 (VBUS_B9)
- new net V3V3_SYS: C201.2, C202.2, R205.2, R206.2, U201.3 (3V3)
- no-connect marks 0 -> 2
Other:
- note added: "BOOT0_RECOVERY / EN_RESET bisher nur Testnetze; physische Jumper/Taster samt Pulls noch zu ergaenzen."
- note added: "GPIO-Budget, weitere Peripherie-Pins und Strap-Pin-Check noch offen. MCU 3.3-V-Versorgung nicht einschalten, bevor die Power-Schaltung fertig ist."
- note added: "TripTracer V1 – ESC MCU/USB: native ESP32-S3 USB2 D-/D+; Quellen-ORing in 03_3V3_USB noch offen."
- note added: "USB-C CC1/CC2 = 5.1k to GND, VBUS -> USB-only power path, USBLC6-2SC6 ESD."
- note removed: "Aktueller Status: PINPLAN UND ELEKTRISCHE VERDRAHTUNG OFFEN."
- note removed: "ESP32-S3-MINI-1-N8 aus V0.3 als Bibliotheksreferenz uebernehmen."
- note removed: "GPIO-Budget erst nach Riverdi-FPC-Belegung endgueltig festlegen."
- note removed: "GPIO0 BOOT Jumper innen, EN/RESET-Service; VBUS-Detektor."
- note removed: "Nativer USB: GPIO19 = D-, GPIO20 = D+. CC1/CC2 je 5.1k Sink, ESD."
- note removed: "V1 ARBEITSBLATT / FUNKTION NOCH NICHT SCHALTPLANMAESSIG UMGESETZT."
- title: TripTracer V1 – ESP32-S3 / USB-Daten / Boot -> TripTracer V1 – ESP32-S3 / native USB-C – Arbeitsstand

Commit message: hardware(esp32): assign GPIO21 timed MCU HOLD and GPIO33 USB-only status
Connections:
- net MCU_HOLD_REQ: now reaches U201.25 (IO21)
- net USB_ACTIVE_N: now reaches U201.28 (IO33)
Other:
- note added: "CONTROL PIN ASSIGNMENTS: U201 GPIO21/pin25 MCU_HOLD_REQ, GPIO33/pin28 USB_ACTIVE_N (TPS2116 ST open drain, requires pullup). Pin budget and strapping final review pending."
Changed lines of the file:
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@@
 (junction (at 387 210.88) (diameter 0) (color 0 0 0 0))
 (junction (at 387 215.96) (diameter 0) (color 0 0 0 0))
+(global_label "MCU_HOLD_REQ" (shape bidirectional) (at 311.42 162.62 0) (effects (font (size 1.0 1.0)) (justify left)))
+(global_label "USB_ACTIVE_N" (shape bidirectional) (at 311.42 177.86 0) (effects (font (size 1.0 1.0)) (justify left)))
+(text "CONTROL PIN ASSIGNMENTS: U201 GPIO21/pin25 MCU_HOLD_REQ, GPIO33/pin28 USB_ACTIVE_N (TPS2116 ST open drain, requires pullup). Pin budget and strapping final review pending." (at 205 55 0) (effects (font (size 1.27 1.27))))
 (sheet_instances (path "/" (page "5"))) (embedded_fonts no)
 )

Commit message: fix(kicad): move symbol terminals and connected labels/wires onto 1.27mm schematic grid
Connections:
- net BOOT0_RECOVERY: no longer U201.4 (IO0)
- net EN_RESET: no longer U201.45 (EN)
- net GND: no longer D201.2 (GND), J201.A1 (GND_A1), J201.A12 (GND_A12), J201.B1 (GND_B1), J201.B12 (GND_B12), J201.SH (SHIELD), U201.1 (GND), U201.2 (GND), U201.42 (GND), U201.43 (GND), U201.46 (GND), U201.47 (GND), U201.48 (GND), U201.49 (GND), U201.50 (GND), U201.51 (GND), U201.52 (GND), U201.53 (GND), U201.54 (GND), U201.55 (GND), U201.56 (GND), U201.57 (GND), U201.58 (GND), U201.59 (GND), U201.60 (GND), U201.61 (GND), U201.62 (GND), U201.63 (GND), U201.64 (GND), U201.65 (GND)
- net MCU_HOLD_REQ: no longer U201.25 (IO21)
- net USB_ACTIVE_N: no longer U201.28 (IO33)
- net USB_DM_MCU: no longer U201.23 (IO19_USB_DM)
- net USB_DM_PORT: no longer D201.3 (IO2_IN), J201.A7 (D-_A7), J201.B7 (D-_B7)
- net USB_DM_PORT_ESD: no longer D201.4 (IO2_OUT)
- net USB_DP_MCU: no longer U201.24 (IO20_USB_DP)
- net USB_DP_PORT: no longer D201.1 (IO1_IN), J201.A6 (D+_A6), J201.B6 (D+_B6)
- net USB_VBUS_RAW: no longer D201.5 (VBUS), J201.A4 (VBUS_A4), J201.A9 (VBUS_A9), J201.B4 (VBUS_B4), J201.B9 (VBUS_B9)
- net V3V3_SYS: no longer U201.3 (3V3)
- net at J201.A5 (CC1): no longer R201.2
- net at J201.B5 (CC2): no longer R202.1
- net at D201.6 (IO1_OUT): no longer R203.1
Other:
- moved on the sheet: C203, D201, J201, R201, R202, R203, R204, R205, R206

Commit message: fix(kicad): revert unsafe bulk ESP32 grid snap that disconnected 3V3 pin
Connections:
- net BOOT0_RECOVERY: now also U201.4 (IO0)
- net EN_RESET: now also U201.45 (EN)
- net GND: now also D201.2 (GND), J201.A1 (GND_A1), J201.A12 (GND_A12), J201.B1 (GND_B1), J201.B12 (GND_B12), J201.SH (SHIELD), U201.1 (GND), U201.2 (GND), U201.42 (GND), U201.43 (GND), U201.46 (GND), U201.47 (GND), U201.48 (GND), U201.49 (GND), U201.50 (GND), U201.51 (GND), U201.52 (GND), U201.53 (GND), U201.54 (GND), U201.55 (GND), U201.56 (GND), U201.57 (GND), U201.58 (GND), U201.59 (GND), U201.60 (GND), U201.61 (GND), U201.62 (GND), U201.63 (GND), U201.64 (GND), U201.65 (GND)
- net MCU_HOLD_REQ: now also U201.25 (IO21)
- net USB_ACTIVE_N: now also U201.28 (IO33)
- net USB_DM_MCU: now also U201.23 (IO19_USB_DM)
- net USB_DM_PORT: now also D201.3 (IO2_IN), J201.A7 (D-_A7), J201.B7 (D-_B7)
- net USB_DM_PORT_ESD: now also D201.4 (IO2_OUT)
- net USB_DP_MCU: now also U201.24 (IO20_USB_DP)
- net USB_DP_PORT: now also D201.1 (IO1_IN), J201.A6 (D+_A6), J201.B6 (D+_B6)
- net USB_VBUS_RAW: now also D201.5 (VBUS), J201.A4 (VBUS_A4), J201.A9 (VBUS_A9), J201.B4 (VBUS_B4), J201.B9 (VBUS_B9)
- net V3V3_SYS: now also U201.3 (3V3)
- net at J201.A5 (CC1): now also R201.2
- net at J201.B5 (CC2): now also R202.1
- net at D201.6 (IO1_OUT): now also R203.1
Other:
- moved on the sheet: C203, D201, J201, R201, R202, R203, R204, R205, R206
