File: hardware/kicad/TripTracer_V1.kicad_pcb (KiCad board)
At the start: 2 copper layers, 21 parts, among them J201 GCT USB4105-GF-A, U101 LMR36520ADDAR 5V/2A CANDIDATE, U201 ESP32-S3-MINI-1-N8

Commit message: fix(kicad): repair LMR38020-Q1 U101 physical PCB pin nets and audit via CI
Parts:
- U101: value LMR36520ADDAR 5V/2A CANDIDATE -> LMR38020SQDDARQ1; footprint Tripmaster:U3_TI_LMR36510ADDAR_DDA -> Tripmaster:TI_LMR38020Q1_DDA_EP
Connections:
- net /5-V-Synchronbuck (elektrischer Entwurf)/BUCK_PGOOD renamed RT_400KHZ
- L101 pad 1: Net-(U101-SW) -> SW_38020
- U101 pad 2: HV_PROTECTED_AFTER_EFUSE -> BUCK_ENABLE
- U101 pad 3: BUCK_ENABLE -> HV_PROTECTED_AFTER_EFUSE
- U101 pad 5: Net-(U101-FB) -> FB_5V
- U101 pad 6: Net-(U101-VCC) -> (no net)
- U101 pad 7: Net-(U101-BOOT) -> BOOT_38020
- U101 pad 8: Net-(U101-SW) -> SW_38020
Changed lines of the file:
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@@
 		)
 	)
-	(footprint "Tripmaster:U3_TI_LMR36510ADDAR_DDA"
+	(footprint "Tripmaster:TI_LMR38020Q1_DDA_EP"
 		(layer "F.Cu")
 		(at 63 52)
-		(descr "TI LMR36510ADDAR PowerPAD DDA0008B, 8+EP9, 5.4mm lead span, EP 2.71x3.4 | Status: HERSTELLER_LANDMASS_EP_MASK_PRUEFEN")
+		(descr "TI LMR38020-Q1 HSOIC DDA0008B provisional, EP 2.71x3.4, manufacturer land/mask review required")
 		(tags "Tripmaster")
 		(property "Reference" "U101"
@@
 			)
 		)
-		(property "Value" "LMR36520ADDAR 5V/2A CANDIDATE"
+		(property "Value" "LMR38020SQDDARQ1"
 			(at 0 4.2 0)
 			(layer "F.Fab")
@@
 			(size 1.55 0.6)
 			(layers "F.Cu" "F.Mask" "F.Paste")
-			(net "HV_PROTECTED_AFTER_EFUSE")
+			(net "BUCK_ENABLE")
 		)
 		(pad "3" smd rect
@@
 			(size 1.55 0.6)
 			(layers "F.Cu" "F.Mask" "F.Paste")
-			(net "BUCK_ENABLE")
+			(net "HV_PROTECTED_AFTER_EFUSE")
 		)
 		(pad "4" smd rect
@@
 			(size 1.55 0.6)
 			(layers "F.Cu" "F.Mask" "F.Paste")
-			(net "/5-V-Synchronbuck (elektrischer Entwurf)/BUCK_PGOOD")
+			(net "RT_400KHZ")
 		)
 		(pad "5" smd rect
@@
 			(size 1.55 0.6)
 			(layers "F.Cu" "F.Mask" "F.Paste")
-			(net "Net-(U101-FB)")
+			(net "FB_5V")
 		)
 		(pad "6" smd rect
@@
 			(size 1.55 0.6)
 			(layers "F.Cu" "F.Mask" "F.Paste")
-			(net "Net-(U101-VCC)")
 		)
 		(pad "7" smd rect
@@
 			(size 1.55 0.6)
 			(layers "F.Cu" "F.Mask" "F.Paste")
-			(net "Net-(U101-BOOT)")
+			(net "BOOT_38020")
 		)
 		(pad "8" smd rect
@@
 			(size 1.55 0.6)
 			(layers "F.Cu" "F.Mask" "F.Paste")
-			(net "Net-(U101-SW)")
+			(net "SW_38020")
 		)
 		(pad "9" smd rect
@@
 			(size 2.15 3.4)
 			(layers "F.Cu" "F.Mask" "F.Paste")
-			(net "Net-(U101-SW)")
+			(net "SW_38020")
 		)
 		(pad "2" smd rect

Commit message: pcb(buck): synchronize L101 15uH FCH, add missing C106/C107/C108/R103, retire C103 VCC and correct net-to-pad parity
Parts:
- removed C103: 1uF VCC, Tripmaster:C_1206_3216
- added C106: 22uF 25V X7R VOUT, Tripmaster:C_1210_3225, F.Cu at (82.0, 55.0)
- added C107: 100nF 100V X7R VIN, Tripmaster:C_1206_3216, F.Cu at (56.0, 49.0)
- added C108: 4.7uF 100V X7R VIN, Tripmaster:C_1210_3225, F.Cu at (49.0, 43.0)
- added R103: 64.9k 1% RT, Tripmaster:R_1206_3216, F.Cu at (52.0, 62.0)
- C102: value 100nF BOOT-SW -> 100nF 100V X7R BOOT-SW
- L101: value 10uH Bourns SRP6030VA-100M (Isat typ 5A) -> 15uH FANGCHENG FCH0650-150M 5.5A Isat; footprint Tripmaster:L_Bourns_SRP6030VA_100M -> Tripmaster:L_FANGCHENG_FCH0650_150M
Connections:
- C101 pad 1: GND -> HV_PROTECTED_AFTER_EFUSE
- C101 pad 2: HV_PROTECTED_AFTER_EFUSE -> GND
- C102 pad 1: Net-(U101-BOOT) -> BOOT_38020
- C102 pad 2: Net-(U101-SW) -> SW_38020
- C104 pad 1: GND -> V5_BUCK_RAW
- C104 pad 2: V5_BUCK_RAW -> GND
- C105 pad 1: GND -> V5_BUCK_RAW
- C105 pad 2: V5_BUCK_RAW -> GND
- R101 pad 1: Net-(U101-FB) -> V5_BUCK_RAW
- R101 pad 2: V5_BUCK_RAW -> FB_5V
- R102 pad 1: GND -> FB_5V
- R102 pad 2: Net-(U101-FB) -> GND

Commit message: pcb: tie U101 EN pad2 to downstream protected VIN pad3 in line with TI absolute maximum ratings
Connections:
- U101 pad 2: BUCK_ENABLE -> HV_PROTECTED_AFTER_EFUSE
Changed lines of the file:
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@@
 			(size 1.55 0.6)
 			(layers "F.Cu" "F.Mask" "F.Paste")
-			(net "BUCK_ENABLE")
+			(net "HV_PROTECTED_AFTER_EFUSE")
 		)
 		(pad "3" smd rect
