File: hardware/modules/TripPower_5V2A/01_Protection_LM74930.kicad_sch (KiCad schematic)
At the start: 38 parts, among them J301 INPUT: VIN/RUN/GND, J302 OUTPUT: VIN_AUX/5V/GND, Q301 STD17NF25 250V CANDIDATE, Q302 BUK7Y4R8-60EX 60V CANDIDATE, U301 LM74930QRGERQ1

Commit message: hardware(TripPower): remove on-module auxiliary fuse F302; expose shared protected VIN_PROTECTED_UNFUSED at J302.1
Parts:
- removed F302: 0997002.WXN 58V 2A + 178.6764.0001 PCB holder, symbol TripPower_Sym:FuseHolder_Mini58V
- J302: value OUTPUT: VIN_AUX/5V/GND -> OUT: PROT_UNFUSED/5V/GND
Connections:
- net VIN_PROTECTED_MAIN is gone; now on net VIN_PROTECTED_UNFUSED: C306.1, R301.2, U301.19 (CS-)
- net VIN_PROTECTED renamed VIN_PROTECTED_UNFUSED
Other:
- note added: "REAL NET-LABEL CONNECTIVITY. SOURCE VIN_FUSED is externally cable-fused. AUX VIN_PROTECTED_UNFUSED IS NOT BRANCH-FUSED ON THIS PCB. LM74930 IS A SHARED ELECTRONIC CIRCUIT BREAKER; EXTERNAL REPLACEABLE BRANCH FUSE AND FAULT-RATED INTERBOARD CONNECTION REQUIRED. KEEP RTN25 FLOAT."
- note added: "STOP GATES: Q301 202V SOA / HOT 2.4A; VS-R313-315 0.75J 350ms; 9V VS BOOT; NO ON-MODULE BRANCH FUSE; EXTERNAL FUSE MANDATORY; J301/J302 POWER; OV/UV/COPPER/ISO. EN DEFAULT: populate R319 only for STANDALONE; TripTracer uses external 3.3V conditioned RUN_CMD."
- note added: "Top: power FETs / controller; below: grouped discrete protection with explicit real nets. INPUT FUSED: J301.1, unfused protected-source VIN_PROTECTED_UNFUSED at J302.1; fuse on TripTracer board as first downstream element, 5V at J302.2."
- note removed: "REAL NET-LABEL CONNECTIVITY. SOURCE VIN_FUSED is externally cable-fused. AUX VIN_PROTECTED is protected through F302 58V MINI; 2A FUSE NOT A GUARANTEED 1A LIMIT. KEEP RTN25 FLOAT."
- note removed: "STOP GATES: Q301 202V SOA / HOT 2.4A; VS-R313-315 0.75J 350ms; 9V VS BOOT; F302 HOLDER FOOTPRINT; J301/J302 POWER; OV/UV/COPPER/ISO. EN DEFAULT: populate R319 only for STANDALONE; TripTracer uses external 3.3V conditioned RUN_CMD."
- note removed: "Top: power FETs / controller; below: grouped discrete protection with explicit real nets. INPUT FUSED: J301.1, output VINPROTECTED via replaceable DC MINI J302.1, 5V after separate LMR38020 sheet J302.2."

Commit message: feat(TripPower): select Vishay 2512 pulse-rated VS resistor candidate and sync stress checks
Parts:
- R313: value 3.32k 200V VS 1 PULSE WIP -> 3.3k 2512 PULSE CANDIDATE; footprint Tripmaster:R_1206_3216 -> Resistor_SMD:R_2512_6332Metric; MPN (none) -> CRCW25123K30FKEGHP
- R314: value 3.32k VS 2 PULSE WIP -> 3.3k 2512 PULSE CANDIDATE; footprint Tripmaster:R_1206_3216 -> Resistor_SMD:R_2512_6332Metric; MPN (none) -> CRCW25123K30FKEGHP
- R315: value 3.32k VS 3 PULSE WIP -> 3.3k 2512 PULSE CANDIDATE; footprint Tripmaster:R_1206_3216 -> Resistor_SMD:R_2512_6332Metric; MPN (none) -> CRCW25123K30FKEGHP
Changed lines of the file:
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@@
 (symbol (lib_id "Tripmaster_Sym:R") (at 405.13 250.19 0) (unit 1) (in_bom yes) (on_board yes) (dnp no) (property "Reference" "R311" (at 405.13 236.22 0) (effects (font (size 1 1)))) (property "Value" "750k UV HIGH 2" (at 405.13 238.76 0) (effects (font (size 1 1)))) (property "Footprint" "Tripmaster:R_1206_3216" (at 405.13 250.19 0) (effects (font (size 1.0 1.0)) (hide yes))) (pin "1") (pin "2") (instances (project "TripPower_5V2A" (path "/f1512578-cc72-4c26-bf70-dbbd00000001/f1512578-cc72-4c26-bf70-dbbd00000002" (reference "R311") (unit 1)))))
 (symbol (lib_id "Tripmaster_Sym:R") (at 490.22 250.19 0) (unit 1) (in_bom yes) (on_board yes) (dnp no) (property "Reference" "R312" (at 490.22 236.22 0) (effects (font (size 1 1)))) (property "Value" "130k UV LOW" (at 490.22 238.76 0) (effects (font (size 1 1)))) (property "Footprint" "Tripmaster:R_1206_3216" (at 490.22 250.19 0) (effects (font (size 1.0 1.0)) (hide yes))) (pin "1") (pin "2") (instances (project "TripPower_5V2A" (path "/f1512578-cc72-4c26-bf70-dbbd00000001/f1512578-cc72-4c26-bf70-dbbd00000002" (reference "R312") (unit 1)))))
-(symbol (lib_id "Tripmaster_Sym:R") (at 64.77 275.59 0) (unit 1) (in_bom yes) (on_board yes) (dnp no) (property "Reference" "R313" (at 64.77 261.62 0) (effects (font (size 1 1)))) (property "Value" "3.32k 200V VS 1 PULSE WIP" (at 64.77 264.16 0) (effects (font (size 1 1)))) (property "Footprint" "Tripmaster:R_1206_3216" (at 64.77 275.59 0) (effects (font (size 1.0 1.0)) (hide yes))) (pin "1") (pin "2") (instances (project "TripPower_5V2A" (path "/f1512578-cc72-4c26-bf70-dbbd00000001/f1512578-cc72-4c26-bf70-dbbd00000002" (reference "R313") (unit 1)))))
-(symbol (lib_id "Tripmaster_Sym:R") (at 149.86 275.59 0) (unit 1) (in_bom yes) (on_board yes) (dnp no) (property "Reference" "R314" (at 149.86 261.62 0) (effects (font (size 1 1)))) (property "Value" "3.32k VS 2 PULSE WIP" (at 149.86 264.16 0) (effects (font (size 1 1)))) (property "Footprint" "Tripmaster:R_1206_3216" (at 149.86 275.59 0) (effects (font (size 1.0 1.0)) (hide yes))) (pin "1") (pin "2") (instances (project "TripPower_5V2A" (path "/f1512578-cc72-4c26-bf70-dbbd00000001/f1512578-cc72-4c26-bf70-dbbd00000002" (reference "R314") (unit 1)))))
-(symbol (lib_id "Tripmaster_Sym:R") (at 234.95 275.59 0) (unit 1) (in_bom yes) (on_board yes) (dnp no) (property "Reference" "R315" (at 234.95 261.62 0) (effects (font (size 1 1)))) (property "Value" "3.32k VS 3 PULSE WIP" (at 234.95 264.16 0) (effects (font (size 1 1)))) (property "Footprint" "Tripmaster:R_1206_3216" (at 234.95 275.59 0) (effects (font (size 1.0 1.0)) (hide yes))) (pin "1") (pin "2") (instances (project "TripPower_5V2A" (path "/f1512578-cc72-4c26-bf70-dbbd00000001/f1512578-cc72-4c26-bf70-dbbd00000002" (reference "R315") (unit 1)))))
+(symbol (lib_id "Tripmaster_Sym:R") (at 64.77 275.59 0) (unit 1) (in_bom yes) (on_board yes) (dnp no) (property "Reference" "R313" (at 64.77 261.62 0) (effects (font (size 1 1)))) (property "Value" "3.3k 2512 PULSE CANDIDATE" (at 64.77 264.16 0) (effects (font (size 1 1)))) (property "Footprint" "Resistor_SMD:R_2512_6332Metric" (at 64.77 275.59 0) (effects (font (size 1.0 1.0)) (hide yes))) (property "MPN" "CRCW25123K30FKEGHP" (at 0 0 0) (effects (font (size 1 1)) (hide yes))) (pin "1") (pin "2") (instances (project "TripPower_5V2A" (path "/f1512578-cc72-4c26-bf70-dbbd00000001/f1512578-cc72-4c26-bf70-dbbd00000002" (reference "R313") (unit 1)))))
+(symbol (lib_id "Tripmaster_Sym:R") (at 149.86 275.59 0) (unit 1) (in_bom yes) (on_board yes) (dnp no) (property "Reference" "R314" (at 149.86 261.62 0) (effects (font (size 1 1)))) (property "Value" "3.3k 2512 PULSE CANDIDATE" (at 149.86 264.16 0) (effects (font (size 1 1)))) (property "Footprint" "Resistor_SMD:R_2512_6332Metric" (at 149.86 275.59 0) (effects (font (size 1.0 1.0)) (hide yes))) (property "MPN" "CRCW25123K30FKEGHP" (at 0 0 0) (effects (font (size 1 1)) (hide yes))) (pin "1") (pin "2") (instances (project "TripPower_5V2A" (path "/f1512578-cc72-4c26-bf70-dbbd00000001/f1512578-cc72-4c26-bf70-dbbd00000002" (reference "R314") (unit 1)))))
+(symbol (lib_id "Tripmaster_Sym:R") (at 234.95 275.59 0) (unit 1) (in_bom yes) (on_board yes) (dnp no) (property "Reference" "R315" (at 234.95 261.62 0) (effects (font (size 1 1)))) (property "Value" "3.3k 2512 PULSE CANDIDATE" (at 234.95 264.16 0) (effects (font (size 1 1)))) (property "Footprint" "Resistor_SMD:R_2512_6332Metric" (at 234.95 275.59 0) (effects (font (size 1.0 1.0)) (hide yes))) (property "MPN" "CRCW25123K30FKEGHP" (at 0 0 0) (effects (font (size 1 1)) (hide yes))) (pin "1") (pin "2") (instances (project "TripPower_5V2A" (path "/f1512578-cc72-4c26-bf70-dbbd00000001/f1512578-cc72-4c26-bf70-dbbd00000002" (reference "R315") (unit 1)))))
 (symbol (lib_id "Tripmaster_Sym:R") (at 320.04 275.59 0) (unit 1) (in_bom yes) (on_board yes) (dnp no) (property "Reference" "R316" (at 320.04 261.62 0) (effects (font (size 1 1)))) (property "Value" "100k EN PULLDOWN" (at 320.04 264.16 0) (effects (font (size 1 1)))) (property "Footprint" "Tripmaster:R_1206_3216" (at 320.04 275.59 0) (effects (font (size 1.0 1.0)) (hide yes))) (pin "1") (pin "2") (instances (project "TripPower_5V2A" (path "/f1512578-cc72-4c26-bf70-dbbd00000001/f1512578-cc72-4c26-bf70-dbbd00000002" (reference "R316") (unit 1)))))
 (symbol (lib_id "Tripmaster_Sym:R") (at 405.13 275.59 0) (unit 1) (in_bom yes) (on_board yes) (dnp no) (property "Reference" "R317" (at 405.13 261.62 0) (effects (font (size 1 1)))) (property "Value" "4.7k RUN SERIES" (at 405.13 264.16 0) (effects (font (size 1 1)))) (property "Footprint" "Tripmaster:R_1206_3216" (at 405.13 275.59 0) (effects (font (size 1.0 1.0)) (hide yes))) (pin "1") (pin "2") (instances (project "TripPower_5V2A" (path "/f1512578-cc72-4c26-bf70-dbbd00000001/f1512578-cc72-4c26-bf70-dbbd00000002" (reference "R317") (unit 1)))))

Commit message: feat(TripPower): select Vishay SQM10250E as Q301 schematic candidate
Parts:
- Q301: value STD17NF25 250V CANDIDATE -> SQM10250E_GE3 250V CANDIDATE; footprint Package_TO_SOT_SMD:TO-252-3_TabPin2 -> Package_TO_SOT_SMD:TO-263-3_TabPin2; MPN (none) -> SQM10250E_GE3
Changed lines of the file:
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@@
  (text "Top: power FETs / controller; below: grouped discrete protection with explicit real nets. INPUT FUSED: J301.1, unfused protected-source VIN_PROTECTED_UNFUSED at J302.1; fuse on TripTracer board as first downstream element, 5V at J302.2." (at 31.75 35.56 0) (effects (font (size 1.27 1.27)) (justify left)))
  (symbol (lib_id "TripTracer_V1:LM74930_Q1_RGE") (at 261.62 132.08 0) (unit 1) (in_bom yes) (on_board yes) (dnp no) (property "Reference" "U301" (at 261.62 118.11 0) (effects (font (size 1 1)))) (property "Value" "LM74930QRGERQ1" (at 261.62 120.65 0) (effects (font (size 1 1)))) (property "Footprint" "Tripmaster:TI_LM74930_RGE0024T_FLOAT_EP" (at 261.62 132.08 0) (effects (font (size 1.0 1.0)) (hide yes))) (pin "1") (pin "2") (pin "3") (pin "4") (pin "5") (pin "6") (pin "7") (pin "8") (pin "9") (pin "10") (pin "11") (pin "12") (pin "13") (pin "14") (pin "15") (pin "16") (pin "17") (pin "18") (pin "19") (pin "20") (pin "21") (pin "22") (pin "23") (pin "24") (pin "25") (instances (project "TripPower_5V2A" (path "/f1512578-cc72-4c26-bf70-dbbd00000001/f1512578-cc72-4c26-bf70-dbbd00000002" (reference "U301") (unit 1)))))
-(symbol (lib_id "TripTracer_V1:PWR_Q_HV") (at 100.33 110.49 0) (unit 1) (in_bom yes) (on_board yes) (dnp no) (property "Reference" "Q301" (at 100.33 96.52 0) (effects (font (size 1 1)))) (property "Value" "STD17NF25 250V CANDIDATE" (at 100.33 99.06 0) (effects (font (size 1 1)))) (property "Footprint" "Package_TO_SOT_SMD:TO-252-3_TabPin2" (at 100.33 110.49 0) (effects (font (size 1.0 1.0)) (hide yes))) (pin "1") (pin "2") (pin "3") (instances (project "TripPower_5V2A" (path "/f1512578-cc72-4c26-bf70-dbbd00000001/f1512578-cc72-4c26-bf70-dbbd00000002" (reference "Q301") (unit 1)))))
+(symbol (lib_id "TripTracer_V1:PWR_Q_HV") (at 100.33 110.49 0) (unit 1) (in_bom yes) (on_board yes) (dnp no) (property "Reference" "Q301" (at 100.33 96.52 0) (effects (font (size 1 1)))) (property "Value" "SQM10250E_GE3 250V CANDIDATE" (at 100.33 99.06 0) (effects (font (size 1 1)))) (property "Footprint" "Package_TO_SOT_SMD:TO-263-3_TabPin2" (at 100.33 110.49 0) (effects (font (size 1.0 1.0)) (hide yes))) (property "MPN" "SQM10250E_GE3" (at 0 0 0) (effects (font (size 1 1)) (hide yes))) (property "Datasheet" "https://www.vishay.com/docs/75035/sqm10250e.pdf" (at 0 0 0) (effects (font (size 1 1)) (hide yes))) (pin "1") (pin "2") (pin "3") (instances (project "TripPower_5V2A" (path "/f1512578-cc72-4c26-bf70-dbbd00000001/f1512578-cc72-4c26-bf70-dbbd00000002" (reference "Q301") (unit 1)))))
 (symbol (lib_id "TripTracer_V1:PWR_Q_LV") (at 431.8 110.49 0) (unit 1) (in_bom yes) (on_board yes) (dnp no) (property "Reference" "Q302" (at 431.8 96.52 0) (effects (font (size 1 1)))) (property "Value" "BUK7Y4R8-60EX 60V CANDIDATE" (at 431.8 99.06 0) (effects (font (size 1 1)))) (property "Footprint" "Package_TO_SOT_SMD:LFPAK56" (at 431.8 110.49 0) (effects (font (size 1.0 1.0)) (hide yes))) (pin "1") (pin "2") (pin "3") (pin "4") (pin "5") (instances (project "TripPower_5V2A" (path "/f1512578-cc72-4c26-bf70-dbbd00000001/f1512578-cc72-4c26-bf70-dbbd00000002" (reference "Q302") (unit 1)))))
 (symbol (lib_id "TripPower_Sym:TripleTerminal") (at 66.04 157.48 0) (unit 1) (in_bom yes) (on_board yes) (dnp no) (property "Reference" "J301" (at 66.04 143.51 0) (effects (font (size 1 1)))) (property "Value" "INPUT: VIN/RUN/GND" (at 66.04 146.05 0) (effects (font (size 1 1)))) (property "Footprint" "Tripmaster:Vehicle_Pigtail_3Wire" (at 66.04 157.48 0) (effects (font (size 1.0 1.0)) (hide yes))) (pin "1") (pin "2") (pin "3") (instances (project "TripPower_5V2A" (path "/f1512578-cc72-4c26-bf70-dbbd00000001/f1512578-cc72-4c26-bf70-dbbd00000002" (reference "J301") (unit 1)))))

Commit message: fix(TripPower): adopt TI HGATE RC dVdt branch instead of series gate resistor
Parts:
- added C307: 10nF 250V dVdt WIP, Tripmaster:C_1206_3216, symbol Tripmaster_Sym:C
- R320: value 100R HGATE SERIES -> 100R dVdt-C SERIES (TI)
Connections:
- net GND: now also C307.2
- net HGATE: now also Q301.1 (G)
- net Q1_GATE renamed DV_DT_RC_NODE
- net DV_DT_RC_NODE: now also C307.1; no longer Q301.1 (G)
Changed lines of the file:
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@@
 (symbol (lib_id "Tripmaster_Sym:R") (at 490.22 275.59 0) (unit 1) (in_bom yes) (on_board yes) (dnp no) (property "Reference" "R318" (at 490.22 261.62 0) (effects (font (size 1 1)))) (property "Value" "100k VS TO AUTO" (at 490.22 264.16 0) (effects (font (size 1 1)))) (property "Footprint" "Tripmaster:R_1206_3216" (at 490.22 275.59 0) (effects (font (size 1.0 1.0)) (hide yes))) (pin "1") (pin "2") (instances (project "TripPower_5V2A" (path "/f1512578-cc72-4c26-bf70-dbbd00000001/f1512578-cc72-4c26-bf70-dbbd00000002" (reference "R318") (unit 1)))))
 (symbol (lib_id "Tripmaster_Sym:R") (at 64.77 299.72 0) (unit 1) (in_bom yes) (on_board yes) (dnp no) (property "Reference" "R319" (at 64.77 285.75 0) (effects (font (size 1 1)))) (property "Value" "0R POPULATE FOR ALWAYS_ON" (at 64.77 288.29 0) (effects (font (size 1 1)))) (property "Footprint" "Tripmaster:R_1206_3216" (at 64.77 299.72 0) (effects (font (size 1.0 1.0)) (hide yes))) (pin "1") (pin "2") (instances (project "TripPower_5V2A" (path "/f1512578-cc72-4c26-bf70-dbbd00000001/f1512578-cc72-4c26-bf70-dbbd00000002" (reference "R319") (unit 1)))))
-(symbol (lib_id "Tripmaster_Sym:R") (at 149.86 299.72 0) (unit 1) (in_bom yes) (on_board yes) (dnp no) (property "Reference" "R320" (at 149.86 285.75 0) (effects (font (size 1 1)))) (property "Value" "100R HGATE SERIES" (at 149.86 288.29 0) (effects (font (size 1 1)))) (property "Footprint" "Tripmaster:R_1206_3216" (at 149.86 299.72 0) (effects (font (size 1.0 1.0)) (hide yes))) (pin "1") (pin "2") (instances (project "TripPower_5V2A" (path "/f1512578-cc72-4c26-bf70-dbbd00000001/f1512578-cc72-4c26-bf70-dbbd00000002" (reference "R320") (unit 1)))))
+(symbol (lib_id "Tripmaster_Sym:R") (at 149.86 299.72 0) (unit 1) (in_bom yes) (on_board yes) (dnp no) (property "Reference" "R320" (at 149.86 285.75 0) (effects (font (size 1 1)))) (property "Value" "100R dVdt-C SERIES (TI)" (at 149.86 288.29 0) (effects (font (size 1 1)))) (property "Footprint" "Tripmaster:R_1206_3216" (at 149.86 299.72 0) (effects (font (size 1.0 1.0)) (hide yes))) (pin "1") (pin "2") (instances (project "TripPower_5V2A" (path "/f1512578-cc72-4c26-bf70-dbbd00000001/f1512578-cc72-4c26-bf70-dbbd00000002" (reference "R320") (unit 1)))))
 (symbol (lib_id "Tripmaster_Sym:C") (at 234.95 299.72 0) (unit 1) (in_bom yes) (on_board yes) (dnp no) (property "Reference" "C301" (at 234.95 285.75 0) (effects (font (size 1 1)))) (property "Value" "47nF 50V TMR" (at 234.95 288.29 0) (effects (font (size 1 1)))) (property "Footprint" "Tripmaster:C_1206_3216" (at 234.95 299.72 0) (effects (font (size 1.0 1.0)) (hide yes))) (pin "1") (pin "2") (instances (project "TripPower_5V2A" (path "/f1512578-cc72-4c26-bf70-dbbd00000001/f1512578-cc72-4c26-bf70-dbbd00000002" (reference "C301") (unit 1)))))
 (symbol (lib_id "Tripmaster_Sym:C") (at 320.04 299.72 0) (unit 1) (in_bom yes) (on_board yes) (dnp no) (property "Reference" "C302" (at 320.04 285.75 0) (effects (font (size 1 1)))) (property "Value" "1uF 100V VS CLAMP" (at 320.04 288.29 0) (effects (font (size 1 1)))) (property "Footprint" "Tripmaster:C_1210_3225" (at 320.04 299.72 0) (effects (font (size 1.0 1.0)) (hide yes))) (pin "1") (pin "2") (instances (project "TripPower_5V2A" (path "/f1512578-cc72-4c26-bf70-dbbd00000001/f1512578-cc72-4c26-bf70-dbbd00000002" (reference "C302") (unit 1)))))
@@
 (global_label "C_NODE" (shape bidirectional) (at 231.14 114.3 0) (effects (font (size 0.9 0.9)) (justify left)))
 (wire (pts (xy 85.09 110.49) (xy 80.01 110.49)) (stroke (width 0) (type default)))
-(global_label "Q1_GATE" (shape bidirectional) (at 80.01 110.49 0) (effects (font (size 0.9 0.9)) (justify left)))
+(global_label "HGATE" (shape bidirectional) (at 80.01 110.49 0) (effects (font (size 0.9 0.9)) (justify left)))
 (wire (pts (xy 115.57 105.41) (xy 120.65 105.41)) (stroke (width 0) (type default)))
 (global_label "VIN_FUSED" (shape bidirectional) (at 120.65 105.41 0) (effects (font (size 0.9 0.9)) (justify left)))
@@
 (global_label "HGATE" (shape bidirectional) (at 133.35 299.72 0) (effects (font (size 0.9 0.9)) (justify left)))
 (wire (pts (xy 161.29 299.72) (xy 166.37 299.72)) (stroke (width 0) (type default)))
-(global_label "Q1_GATE" (shape bidirectional) (at 166.37 299.72 0) (effects (font (size 0.9 0.9)) (justify left)))
+(global_label "DV_DT_RC_NODE" (shape bidirectional) (at 166.37 299.72 0) (effects (font (size 0.9 0.9)) (justify left)))
 (wire (pts (xy 223.52 299.72) (xy 218.44 299.72)) (stroke (width 0) (type default)))
 (global_label "TMR_NODE" (shape bidirectional) (at 218.44 299.72 0) (effects (font (size 0.9 0.9)) (justify left)))
@@
 (wire (pts (xy 161.29 400.05) (xy 166.37 400.05)) (stroke (width 0) (type default)))
 (global_label "RUN_ISOLATED_AFTER_R" (shape bidirectional) (at 166.37 400.05 0) (effects (font (size 0.9 0.9)) (justify left)))
+(symbol (lib_id "Tripmaster_Sym:C") (at 149.86 350.52 0) (unit 1) (in_bom yes) (on_board yes) (dnp no) (property "Reference" "C307" (at 149.86 336.55 0) (effects (font (size 1 1)))) (property "Value" "10nF 250V dVdt WIP" (at 149.86 339.09 0) (effects (font (size 1 1)))) (property "Footprint" "Tripmaster:C_1206_3216" (at 149.86 350.52 0) (effects (font (size 1.0 1.0)) (hide yes))) (property "MPN" "C1206C103JARECAUTO" (at 0 0 0) (effects (font (size 1 1)) (hide yes))) (property "Datasheet" "https://www.digikey.de/en/products/detail/kemet/C1206C103JARECAUTO/16680107" (at 0 0 0) (effects (font (size 1 1)) (hide yes))) (pin "1") (pin "2") (instances (project "TripPower_5V2A" (path "/f1512578-cc72-4c26-bf70-dbbd00000001/f1512578-cc72-4c26-bf70-dbbd00000002" (reference "C307") (unit 1)))))
+(wire (pts (xy 138.43 350.52) (xy 133.35 350.52)) (stroke (width 0) (type default)))
+(global_label "DV_DT_RC_NODE" (shape bidirectional) (at 133.35 350.52 0) (effects (font (size 0.9 0.9)) (justify left)))
+(wire (pts (xy 161.29 350.52) (xy 166.37 350.52)) (stroke (width 0) (type default)))
+(global_label "GND" (shape bidirectional) (at 166.37 350.52 0) (effects (font (size 0.9 0.9)) (justify left)))
  (embedded_fonts no))
