File: hardware/modules/TripPower_5V2A/01_Protection_LM74930.kicad_sch (KiCad schematic)
At the start: 40 parts, among them J301 INPUT: VIN/RUN/GND, J302 OUT: PROT_UNFUSED/5V/GND, Q301 SQM10250E_GE3 250V CANDIDATE, Q302 BUK7Y4R8-60EX 60V CANDIDATE, U301 LM74930QRGERQ1

Commit message: feat(TripPower): implement RESET-qualified AUTO/RUN series EN interlock with automotive MOSFET, clamps and C309 DNP
Parts:
- C309: Status AUTO_EN_ONLY; RUN_CMD bypass not yet gated -> DNP; supervisor U302 controls Q303 series enable, no RC del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; now not fitted
- R316: value 100k EN PULLDOWN -> 5.6k EN PULLDOWN / VS_READY GATE
- R318: value 100k VS TO AUTO -> 22k VS TO AUTO_REQ (GATED)
Connections:
- net CTRL_EN: no longer D305.1 (K), R319.2
- new net EN_REQUEST_RAW: D305.1 (K), R319.2
Changed lines of the file:
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@@
 (symbol (lib_id "Tripmaster_Sym:R") (at 149.86 275.59 0) (unit 1) (in_bom yes) (on_board yes) (dnp no) (property "Reference" "R314" (at 149.86 261.62 0) (effects (font (size 1 1)))) (property "Value" "3.3k 2512 PULSE CANDIDATE" (at 149.86 264.16 0) (effects (font (size 1 1)))) (property "Footprint" "Resistor_SMD:R_2512_6332Metric" (at 149.86 275.59 0) (effects (font (size 1.0 1.0)) (hide yes))) (property "MPN" "CRCW25123K30FKEGHP" (at 0 0 0) (effects (font (size 1 1)) (hide yes))) (pin "1") (pin "2") (instances (project "TripPower_5V2A" (path "/f1512578-cc72-4c26-bf70-dbbd00000001/f1512578-cc72-4c26-bf70-dbbd00000002" (reference "R314") (unit 1)))))
 (symbol (lib_id "Tripmaster_Sym:R") (at 234.95 275.59 0) (unit 1) (in_bom yes) (on_board yes) (dnp no) (property "Reference" "R315" (at 234.95 261.62 0) (effects (font (size 1 1)))) (property "Value" "3.3k 2512 PULSE CANDIDATE" (at 234.95 264.16 0) (effects (font (size 1 1)))) (property "Footprint" "Resistor_SMD:R_2512_6332Metric" (at 234.95 275.59 0) (effects (font (size 1.0 1.0)) (hide yes))) (property "MPN" "CRCW25123K30FKEGHP" (at 0 0 0) (effects (font (size 1 1)) (hide yes))) (pin "1") (pin "2") (instances (project "TripPower_5V2A" (path "/f1512578-cc72-4c26-bf70-dbbd00000001/f1512578-cc72-4c26-bf70-dbbd00000002" (reference "R315") (unit 1)))))
-(symbol (lib_id "Tripmaster_Sym:R") (at 320.04 275.59 0) (unit 1) (in_bom yes) (on_board yes) (dnp no) (property "Reference" "R316" (at 320.04 261.62 0) (effects (font (size 1 1)))) (property "Value" "100k EN PULLDOWN" (at 320.04 264.16 0) (effects (font (size 1 1)))) (property "Footprint" "Tripmaster:R_1206_3216" (at 320.04 275.59 0) (effects (font (size 1.0 1.0)) (hide yes))) (pin "1") (pin "2") (instances (project "TripPower_5V2A" (path "/f1512578-cc72-4c26-bf70-dbbd00000001/f1512578-cc72-4c26-bf70-dbbd00000002" (reference "R316") (unit 1)))))
+(symbol (lib_id "Tripmaster_Sym:R") (at 320.04 275.59 0) (unit 1) (in_bom yes) (on_board yes) (dnp no) (property "Reference" "R316" (at 320.04 261.62 0) (effects (font (size 1 1)))) (property "Value" "5.6k EN PULLDOWN / VS_READY GATE" (at 320.04 264.16 0) (effects (font (size 1 1)))) (property "Footprint" "Tripmaster:R_1206_3216" (at 320.04 275.59 0) (effects (font (size 1.0 1.0)) (hide yes))) (pin "1") (pin "2") (instances (project "TripPower_5V2A" (path "/f1512578-cc72-4c26-bf70-dbbd00000001/f1512578-cc72-4c26-bf70-dbbd00000002" (reference "R316") (unit 1)))))
 (symbol (lib_id "Tripmaster_Sym:R") (at 405.13 275.59 0) (unit 1) (in_bom yes) (on_board yes) (dnp no) (property "Reference" "R317" (at 405.13 261.62 0) (effects (font (size 1 1)))) (property "Value" "4.7k RUN SERIES" (at 405.13 264.16 0) (effects (font (size 1 1)))) (property "Footprint" "Tripmaster:R_1206_3216" (at 405.13 275.59 0) (effects (font (size 1.0 1.0)) (hide yes))) (pin "1") (pin "2") (instances (project "TripPower_5V2A" (path "/f1512578-cc72-4c26-bf70-dbbd00000001/f1512578-cc72-4c26-bf70-dbbd00000002" (reference "R317") (unit 1)))))
-(symbol (lib_id "Tripmaster_Sym:R") (at 490.22 275.59 0) (unit 1) (in_bom yes) (on_board yes) (dnp no) (property "Reference" "R318" (at 490.22 261.62 0) (effects (font (size 1 1)))) (property "Value" "100k VS TO AUTO" (at 490.22 264.16 0) (effects (font (size 1 1)))) (property "Footprint" "Tripmaster:R_1206_3216" (at 490.22 275.59 0) (effects (font (size 1.0 1.0)) (hide yes))) (pin "1") (pin "2") (instances (project "TripPower_5V2A" (path "/f1512578-cc72-4c26-bf70-dbbd00000001/f1512578-cc72-4c26-bf70-dbbd00000002" (reference "R318") (unit 1)))))
+(symbol (lib_id "Tripmaster_Sym:R") (at 490.22 275.59 0) (unit 1) (in_bom yes) (on_board yes) (dnp no) (property "Reference" "R318" (at 490.22 261.62 0) (effects (font (size 1 1)))) (property "Value" "22k VS TO AUTO_REQ (GATED)" (at 490.22 264.16 0) (effects (font (size 1 1)))) (property "Footprint" "Tripmaster:R_1206_3216" (at 490.22 275.59 0) (effects (font (size 1.0 1.0)) (hide yes))) (pin "1") (pin "2") (instances (project "TripPower_5V2A" (path "/f1512578-cc72-4c26-bf70-dbbd00000001/f1512578-cc72-4c26-bf70-dbbd00000002" (reference "R318") (unit 1)))))
 (symbol (lib_id "Tripmaster_Sym:R") (at 64.77 299.72 0) (unit 1) (in_bom yes) (on_board yes) (dnp no) (property "Reference" "R319" (at 64.77 285.75 0) (effects (font (size 1 1)))) (property "Value" "0R POPULATE FOR ALWAYS_ON" (at 64.77 288.29 0) (effects (font (size 1 1)))) (property "Footprint" "Tripmaster:R_1206_3216" (at 64.77 299.72 0) (effects (font (size 1.0 1.0)) (hide yes))) (pin "1") (pin "2") (instances (project "TripPower_5V2A" (path "/f1512578-cc72-4c26-bf70-dbbd00000001/f1512578-cc72-4c26-bf70-dbbd00000002" (reference "R319") (unit 1)))))
 (symbol (lib_id "Tripmaster_Sym:R") (at 149.86 299.72 0) (unit 1) (in_bom yes) (on_board yes) (dnp no) (property "Reference" "R320" (at 149.86 285.75 0) (effects (font (size 1 1)))) (property "Value" "100R dVdt-C SERIES (TI)" (at 149.86 288.29 0) (effects (font (size 1 1)))) (property "Footprint" "Tripmaster:R_1206_3216" (at 149.86 299.72 0) (effects (font (size 1.0 1.0)) (hide yes))) (pin "1") (pin "2") (instances (project "TripPower_5V2A" (path "/f1512578-cc72-4c26-bf70-dbbd00000001/f1512578-cc72-4c26-bf70-dbbd00000002" (reference "R320") (unit 1)))))
@@
 (global_label "AUTO_EN_LINK" (shape bidirectional) (at 48.26 299.72 0) (effects (font (size 0.9 0.9)) (justify left)))
 (wire (pts (xy 76.2 299.72) (xy 81.28 299.72)) (stroke (width 0) (type default)))
-(global_label "CTRL_EN" (shape bidirectional) (at 81.28 299.72 0) (effects (font (size 0.9 0.9)) (justify left)))
+(global_label "EN_REQUEST_RAW" (shape bidirectional) (at 81.28 299.72 0) (effects (font (size 0.9 0.9)) (justify left)))
 (wire (pts (xy 138.43 299.72) (xy 133.35 299.72)) (stroke (width 0) (type default)))
 (global_label "HGATE" (shape bidirectional) (at 133.35 299.72 0) (effects (font (size 0.9 0.9)) (justify left)))
@@
 (instances (project "TripPower_5V2A" (path "/f1512578-cc72-4c26-bf70-dbbd00000001/f1512578-cc72-4c26-bf70-dbbd00000002" (reference "D305") (unit 1)))))
 (wire (pts (xy 140.97 400.05) (xy 135.89 400.05)) (stroke (width 0) (type default)))
-(global_label "CTRL_EN" (shape bidirectional) (at 135.89 400.05 0) (effects (font (size 0.9 0.9)) (justify left)))
+(global_label "EN_REQUEST_RAW" (shape bidirectional) (at 135.89 400.05 0) (effects (font (size 0.9 0.9)) (justify left)))
 (wire (pts (xy 161.29 400.05) (xy 166.37 400.05)) (stroke (width 0) (type default)))
 (global_label "RUN_ISOLATED_AFTER_R" (shape bidirectional) (at 166.37 400.05 0) (effects (font (size 0.9 0.9)) (justify left)))
@@
 (wire (pts (xy 330.2 350.52) (xy 336.55 350.52)) (stroke (width 0) (type default)))
 (global_label "GND" (shape bidirectional) (at 336.55 350.52 0) (effects (font (size 0.9 0.9)) (justify left)))
-(symbol (lib_id "Tripmaster_Sym:C") (at 405.13 350.52 0) (unit 1) (in_bom yes) (on_board yes) (dnp no) (property "Reference" "C309" (at 405.13 336.55 0) (effects (font (size 1 1)))) (property "Value" "10uF 50V EN DELAY WIP" (at 405.13 339.09 0) (effects (font (size 1 1)))) (property "Footprint" "Capacitor_SMD:C_1210_3225Metric" (at 405.13 350.52 0) (effects (font (size 1.0 1.0)) (hide yes))) (property "MPN" "12105C106K4T2A" (at 0 0 0) (effects (font (size 1 1)) (hide yes))) (property "Supplier_URL" "https://www.mouser.de/de/ProductDetail/KEMET/12105C106K4T2A" (at 0 0 0) (effects (font (size 1 1)) (hide yes))) (property "Status" "AUTO_EN_ONLY; RUN_CMD bypass not yet gated" (at 0 0 0) (effects (font (size 1 1)) (hide yes))) (pin "1") (pin "2") (instances (project "TripPower_5V2A" (path "/f1512578-cc72-4c26-bf70-dbbd00000001/f1512578-cc72-4c26-bf70-dbbd00000002" (reference "C309") (unit 1)))))
+(symbol (lib_id "Tripmaster_Sym:C") (at 405.13 350.52 0) (unit 1) (in_bom yes) (on_board yes) (dnp yes) (property "Reference" "C309" (at 405.13 336.55 0) (effects (font (size 1 1)))) (property "Value" "10uF 50V EN DELAY WIP" (at 405.13 339.09 0) (effects (font (size 1 1)))) (property "Footprint" "Capacitor_SMD:C_1210_3225Metric" (at 405.13 350.52 0) (effects (font (size 1.0 1.0)) (hide yes))) (property "MPN" "12105C106K4T2A" (at 0 0 0) (effects (font (size 1 1)) (hide yes))) (property "Supplier_URL" "https://www.mouser.de/de/ProductDetail/KEMET/12105C106K4T2A" (at 0 0 0) (effects (font (size 1 1)) (hide yes))) (property "Status" "DNP; supervisor U302 controls Q303 series enable, no RC delay" (at 0 0 0) (effects (font (size 1 1)) (hide yes))) (pin "1") (pin "2") (instances (project "TripPower_5V2A" (path "/f1512578-cc72-4c26-bf70-dbbd00000001/f1512578-cc72-4c26-bf70-dbbd00000002" (reference "C309") (unit 1)))))
 (wire (pts (xy 393.7 350.52) (xy 388.62 350.52)) (stroke (width 0) (type default)))
 (global_label "CTRL_EN" (shape bidirectional) (at 388.62 350.52 0) (effects (font (size 0.9 0.9)) (justify left)))

Commit message: feat(TripPower): replace leaking EN source follower with VS-only 300V automotive PNP/NPN gated high-side drive; isolate RUN and AUTO
Parts:
- D305: now not fitted
- R316: value 5.6k EN PULLDOWN / VS_READY GATE -> 33k EN PULLDOWN - NEW HIGH-SIDE PNP
- R318: value 22k VS TO AUTO_REQ (GATED) -> 100k PNP OUTPUT TO EN
Connections:
- net CTRL_EN: now also R318.2
- net GND: now also R319.2
- net VS_CLAMP: no longer R318.1
- net AUTO_EN_LINK renamed RUN_BYPASS_NODE
- net RUN_BYPASS_NODE: no longer R318.2
- net EN_REQUEST_RAW renamed DNP_RUN_PATH
- net DNP_RUN_PATH: no longer R319.2
- net RUN_ISOLATED_AFTER_R renamed DNP_RUN_SERIES
- net DNP_RUN_SERIES: no longer R317.2
- new net PNP_OUT: R318.1
- new net RUN_BASE: R317.2
Changed lines of the file:
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@@
 (symbol (lib_id "Tripmaster_Sym:R") (at 149.86 275.59 0) (unit 1) (in_bom yes) (on_board yes) (dnp no) (property "Reference" "R314" (at 149.86 261.62 0) (effects (font (size 1 1)))) (property "Value" "3.3k 2512 PULSE CANDIDATE" (at 149.86 264.16 0) (effects (font (size 1 1)))) (property "Footprint" "Resistor_SMD:R_2512_6332Metric" (at 149.86 275.59 0) (effects (font (size 1.0 1.0)) (hide yes))) (property "MPN" "CRCW25123K30FKEGHP" (at 0 0 0) (effects (font (size 1 1)) (hide yes))) (pin "1") (pin "2") (instances (project "TripPower_5V2A" (path "/f1512578-cc72-4c26-bf70-dbbd00000001/f1512578-cc72-4c26-bf70-dbbd00000002" (reference "R314") (unit 1)))))
 (symbol (lib_id "Tripmaster_Sym:R") (at 234.95 275.59 0) (unit 1) (in_bom yes) (on_board yes) (dnp no) (property "Reference" "R315" (at 234.95 261.62 0) (effects (font (size 1 1)))) (property "Value" "3.3k 2512 PULSE CANDIDATE" (at 234.95 264.16 0) (effects (font (size 1 1)))) (property "Footprint" "Resistor_SMD:R_2512_6332Metric" (at 234.95 275.59 0) (effects (font (size 1.0 1.0)) (hide yes))) (property "MPN" "CRCW25123K30FKEGHP" (at 0 0 0) (effects (font (size 1 1)) (hide yes))) (pin "1") (pin "2") (instances (project "TripPower_5V2A" (path "/f1512578-cc72-4c26-bf70-dbbd00000001/f1512578-cc72-4c26-bf70-dbbd00000002" (reference "R315") (unit 1)))))
-(symbol (lib_id "Tripmaster_Sym:R") (at 320.04 275.59 0) (unit 1) (in_bom yes) (on_board yes) (dnp no) (property "Reference" "R316" (at 320.04 261.62 0) (effects (font (size 1 1)))) (property "Value" "5.6k EN PULLDOWN / VS_READY GATE" (at 320.04 264.16 0) (effects (font (size 1 1)))) (property "Footprint" "Tripmaster:R_1206_3216" (at 320.04 275.59 0) (effects (font (size 1.0 1.0)) (hide yes))) (pin "1") (pin "2") (instances (project "TripPower_5V2A" (path "/f1512578-cc72-4c26-bf70-dbbd00000001/f1512578-cc72-4c26-bf70-dbbd00000002" (reference "R316") (unit 1)))))
+(symbol (lib_id "Tripmaster_Sym:R") (at 320.04 275.59 0) (unit 1) (in_bom yes) (on_board yes) (dnp no) (property "Reference" "R316" (at 320.04 261.62 0) (effects (font (size 1 1)))) (property "Value" "33k EN PULLDOWN - NEW HIGH-SIDE PNP" (at 320.04 264.16 0) (effects (font (size 1 1)))) (property "Footprint" "Tripmaster:R_1206_3216" (at 320.04 275.59 0) (effects (font (size 1.0 1.0)) (hide yes))) (pin "1") (pin "2") (instances (project "TripPower_5V2A" (path "/f1512578-cc72-4c26-bf70-dbbd00000001/f1512578-cc72-4c26-bf70-dbbd00000002" (reference "R316") (unit 1)))))
 (symbol (lib_id "Tripmaster_Sym:R") (at 405.13 275.59 0) (unit 1) (in_bom yes) (on_board yes) (dnp no) (property "Reference" "R317" (at 405.13 261.62 0) (effects (font (size 1 1)))) (property "Value" "4.7k RUN SERIES" (at 405.13 264.16 0) (effects (font (size 1 1)))) (property "Footprint" "Tripmaster:R_1206_3216" (at 405.13 275.59 0) (effects (font (size 1.0 1.0)) (hide yes))) (pin "1") (pin "2") (instances (project "TripPower_5V2A" (path "/f1512578-cc72-4c26-bf70-dbbd00000001/f1512578-cc72-4c26-bf70-dbbd00000002" (reference "R317") (unit 1)))))
-(symbol (lib_id "Tripmaster_Sym:R") (at 490.22 275.59 0) (unit 1) (in_bom yes) (on_board yes) (dnp no) (property "Reference" "R318" (at 490.22 261.62 0) (effects (font (size 1 1)))) (property "Value" "22k VS TO AUTO_REQ (GATED)" (at 490.22 264.16 0) (effects (font (size 1 1)))) (property "Footprint" "Tripmaster:R_1206_3216" (at 490.22 275.59 0) (effects (font (size 1.0 1.0)) (hide yes))) (pin "1") (pin "2") (instances (project "TripPower_5V2A" (path "/f1512578-cc72-4c26-bf70-dbbd00000001/f1512578-cc72-4c26-bf70-dbbd00000002" (reference "R318") (unit 1)))))
+(symbol (lib_id "Tripmaster_Sym:R") (at 490.22 275.59 0) (unit 1) (in_bom yes) (on_board yes) (dnp no) (property "Reference" "R318" (at 490.22 261.62 0) (effects (font (size 1 1)))) (property "Value" "100k PNP OUTPUT TO EN" (at 490.22 264.16 0) (effects (font (size 1 1)))) (property "Footprint" "Tripmaster:R_1206_3216" (at 490.22 275.59 0) (effects (font (size 1.0 1.0)) (hide yes))) (pin "1") (pin "2") (instances (project "TripPower_5V2A" (path "/f1512578-cc72-4c26-bf70-dbbd00000001/f1512578-cc72-4c26-bf70-dbbd00000002" (reference "R318") (unit 1)))))
 (symbol (lib_id "Tripmaster_Sym:R") (at 64.77 299.72 0) (unit 1) (in_bom yes) (on_board yes) (dnp no) (property "Reference" "R319" (at 64.77 285.75 0) (effects (font (size 1 1)))) (property "Value" "0R POPULATE FOR ALWAYS_ON" (at 64.77 288.29 0) (effects (font (size 1 1)))) (property "Footprint" "Tripmaster:R_1206_3216" (at 64.77 299.72 0) (effects (font (size 1.0 1.0)) (hide yes))) (pin "1") (pin "2") (instances (project "TripPower_5V2A" (path "/f1512578-cc72-4c26-bf70-dbbd00000001/f1512578-cc72-4c26-bf70-dbbd00000002" (reference "R319") (unit 1)))))
 (symbol (lib_id "Tripmaster_Sym:R") (at 149.86 299.72 0) (unit 1) (in_bom yes) (on_board yes) (dnp no) (property "Reference" "R320" (at 149.86 285.75 0) (effects (font (size 1 1)))) (property "Value" "100R dVdt-C SERIES (TI)" (at 149.86 288.29 0) (effects (font (size 1 1)))) (property "Footprint" "Tripmaster:R_1206_3216" (at 149.86 299.72 0) (effects (font (size 1.0 1.0)) (hide yes))) (pin "1") (pin "2") (instances (project "TripPower_5V2A" (path "/f1512578-cc72-4c26-bf70-dbbd00000001/f1512578-cc72-4c26-bf70-dbbd00000002" (reference "R320") (unit 1)))))
@@
 (global_label "RUN_CMD" (shape bidirectional) (at 388.62 275.59 0) (effects (font (size 0.9 0.9)) (justify left)))
 (wire (pts (xy 416.56 275.59) (xy 421.64 275.59)) (stroke (width 0) (type default)))
-(global_label "RUN_ISOLATED_AFTER_R" (shape bidirectional) (at 421.64 275.59 0) (effects (font (size 0.9 0.9)) (justify left)))
+(global_label "RUN_BASE" (shape bidirectional) (at 421.64 275.59 0) (effects (font (size 0.9 0.9)) (justify left)))
 (wire (pts (xy 478.79 275.59) (xy 473.71 275.59)) (stroke (width 0) (type default)))
-(global_label "VS_CLAMP" (shape bidirectional) (at 473.71 275.59 0) (effects (font (size 0.9 0.9)) (justify left)))
+(global_label "PNP_OUT" (shape bidirectional) (at 473.71 275.59 0) (effects (font (size 0.9 0.9)) (justify left)))
 (wire (pts (xy 501.65 275.59) (xy 506.73 275.59)) (stroke (width 0) (type default)))
-(global_label "AUTO_EN_LINK" (shape bidirectional) (at 506.73 275.59 0) (effects (font (size 0.9 0.9)) (justify left)))
+(global_label "CTRL_EN" (shape bidirectional) (at 506.73 275.59 0) (effects (font (size 0.9 0.9)) (justify left)))
 (wire (pts (xy 53.34 299.72) (xy 48.26 299.72)) (stroke (width 0) (type default)))
-(global_label "AUTO_EN_LINK" (shape bidirectional) (at 48.26 299.72 0) (effects (font (size 0.9 0.9)) (justify left)))
+(global_label "RUN_BYPASS_NODE" (shape bidirectional) (at 48.26 299.72 0) (effects (font (size 0.9 0.9)) (justify left)))
 (wire (pts (xy 76.2 299.72) (xy 81.28 299.72)) (stroke (width 0) (type default)))
-(global_label "EN_REQUEST_RAW" (shape bidirectional) (at 81.28 299.72 0) (effects (font (size 0.9 0.9)) (justify left)))
+(global_label "GND" (shape bidirectional) (at 81.28 299.72 0) (effects (font (size 0.9 0.9)) (justify left)))
 (wire (pts (xy 138.43 299.72) (xy 133.35 299.72)) (stroke (width 0) (type default)))
 (global_label "HGATE" (shape bidirectional) (at 133.35 299.72 0) (effects (font (size 0.9 0.9)) (justify left)))
@@
 (global_label "FAULT_OC_N" (shape bidirectional) (at 48.26 400.05 0) (effects (font (size 0.9 0.9)) (justify left)))
 (global_label "5V_OUT" (shape bidirectional) (at 81.28 400.05 0) (effects (font (size 0.9 0.9)) (justify left)))
-(symbol (lib_id "TripTracer_V1:PWR_DIODE") (at 151.13 400.05 0) (unit 1) (in_bom yes) (on_board yes) (dnp no)
+(symbol (lib_id "TripTracer_V1:PWR_DIODE") (at 151.13 400.05 0) (unit 1) (in_bom yes) (on_board yes) (dnp yes)
 (property "Reference" "D305" (at 151.13 384.81 0) (effects (font (size 1 1))))
 (property "Value" "BAS116Q-7-F LOW_LEAK RUN BLOCK" (at 151.13 388.62 0) (effects (font (size 1 1))))
@@
 (instances (project "TripPower_5V2A" (path "/f1512578-cc72-4c26-bf70-dbbd00000001/f1512578-cc72-4c26-bf70-dbbd00000002" (reference "D305") (unit 1)))))
 (wire (pts (xy 140.97 400.05) (xy 135.89 400.05)) (stroke (width 0) (type default)))
-(global_label "EN_REQUEST_RAW" (shape bidirectional) (at 135.89 400.05 0) (effects (font (size 0.9 0.9)) (justify left)))
+(global_label "DNP_RUN_PATH" (shape bidirectional) (at 135.89 400.05 0) (effects (font (size 0.9 0.9)) (justify left)))
 (wire (pts (xy 161.29 400.05) (xy 166.37 400.05)) (stroke (width 0) (type default)))
-(global_label "RUN_ISOLATED_AFTER_R" (shape bidirectional) (at 166.37 400.05 0) (effects (font (size 0.9 0.9)) (justify left)))
+(global_label "DNP_RUN_SERIES" (shape bidirectional) (at 166.37 400.05 0) (effects (font (size 0.9 0.9)) (justify left)))
 (symbol (lib_id "Tripmaster_Sym:C") (at 149.86 350.52 0) (unit 1) (in_bom yes) (on_board yes) (dnp no) (property "Reference" "C307" (at 149.86 336.55 0) (effects (font (size 1 1)))) (property "Value" "10nF 250V dVdt WIP" (at 149.86 339.09 0) (effects (font (size 1 1)))) (property "Footprint" "Tripmaster:C_1206_3216" (at 149.86 350.52 0) (effects (font (size 1.0 1.0)) (hide yes))) (property "MPN" "C1206C103JARECAUTO" (at 0 0 0) (effects (font (size 1 1)) (hide yes))) (property "Datasheet" "https://www.digikey.de/en/products/detail/kemet/C1206C103JARECAUTO/16680107" (at 0 0 0) (effects (font (size 1 1)) (hide yes))) (pin "1") (pin "2") (instances (project "TripPower_5V2A" (path "/f1512578-cc72-4c26-bf70-dbbd00000001/f1512578-cc72-4c26-bf70-dbbd00000002" (reference "C307") (unit 1)))))
 (wire (pts (xy 138.43 350.52) (xy 133.35 350.52)) (stroke (width 0) (type default)))
