File: hardware/modules/TripPower_5V2A/01_Protection_LM74930.kicad_sch (KiCad schematic)
At the start: 40 parts, among them J301 INPUT: VIN/RUN/GND, J302 OUT: PROT_UNFUSED/5V/GND, Q301 SQM10250E_GE3 250V CANDIDATE, Q302 BUK7Y4R8-60EX 60V CANDIDATE, U301 LM74930QRGERQ1

Commit message: feat(TripPower REV4): add second 10uF 100V automotive ceramic C312 VS hold-up in parallel
Parts:
- added C312: 10uF 100V VS STARTUP RESERVOIR X7R REV4, Capacitor_SMD:C_2220_5750Metric, symbol Tripmaster_Sym:C
Connections:
- net GND: now also C312.2
- net VS_CLAMP: now also C312.1
Changed lines of the file:
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@@
 (wire (pts (xy 331.47 350.52) (xy 336.55 350.52)) (stroke (width 0) (type default)))
 (global_label "GND" (shape bidirectional) (at 336.55 350.52 0) (effects (font (size 0.9 0.9)) (justify left)))
+(symbol (lib_id "Tripmaster_Sym:C") (at 490.22 350.52 0) (unit 1) (in_bom yes) (on_board yes) (dnp no) (property "Reference" "C312" (at 490.22 336.55 0) (effects (font (size 1 1)))) (property "Value" "10uF 100V VS STARTUP RESERVOIR X7R REV4" (at 490.22 339.09 0) (effects (font (size 1 1)))) (property "Footprint" "Capacitor_SMD:C_2220_5750Metric" (at 490.22 350.52 0) (effects (font (size 1.0 1.0)) (hide yes))) (property "MPN" "KAF55CR72A106KV" (at 0 0 0) (effects (font (size 1 1)) (hide yes))) (property "Supplier_URL" "https://www.mouser.de/de/ProductDetail/KYOCERA-AVX/KAF55CR72A106KV" (at 0 0 0) (effects (font (size 1 1)) (hide yes))) (pin "1") (pin "2") (instances (project "TripPower_5V2A" (path "/f1512578-cc72-4c26-bf70-dbbd00000001/f1512578-cc72-4c26-bf70-dbbd00000002" (reference "C312") (unit 1)))))
+(wire (pts (xy 478.79 350.52) (xy 473.71 350.52)) (stroke (width 0) (type default)))
+(global_label "VS_CLAMP" (shape bidirectional) (at 473.71 350.52 0) (effects (font (size 0.9 0.9)) (justify left)))
+(wire (pts (xy 501.65 350.52) (xy 506.73 350.52)) (stroke (width 0) (type default)))
+(global_label "GND" (shape bidirectional) (at 506.73 350.52 0) (effects (font (size 0.9 0.9)) (justify left)))
 (symbol (lib_id "Tripmaster_Sym:C") (at 405.13 350.52 0) (unit 1) (in_bom yes) (on_board yes) (dnp yes) (property "Reference" "C309" (at 405.13 336.55 0) (effects (font (size 1 1)))) (property "Value" "10uF 50V EN DELAY WIP" (at 405.13 339.09 0) (effects (font (size 1 1)))) (property "Footprint" "Capacitor_SMD:C_1210_3225Metric" (at 405.13 350.52 0) (effects (font (size 1.0 1.0)) (hide yes))) (property "MPN" "12105C106K4T2A" (at 0 0 0) (effects (font (size 1 1)) (hide yes))) (property "Supplier_URL" "https://www.mouser.de/de/ProductDetail/KEMET/12105C106K4T2A" (at 0 0 0) (effects (font (size 1 1)) (hide yes))) (property "Status" "DNP; supervisor U302 controls Q303 series enable, no RC delay" (at 0 0 0) (effects (font (size 1 1)) (hide yes))) (pin "1") (pin "2") (instances (project "TripPower_5V2A" (path "/f1512578-cc72-4c26-bf70-dbbd00000001/f1512578-cc72-4c26-bf70-dbbd00000002" (reference "C309") (unit 1)))))
 (wire (pts (xy 393.7 350.52) (xy 388.62 350.52)) (stroke (width 0) (type default)))

Commit message: fix(TripPower): lock verified automotive 1uF/100V VS/A bypass and 100nF/250V VIN MLCC MPNs; correct C304 1210 footprint
Parts:
- C302: MPN (none) -> C1210C105K1RACAUTO; Supplier_URL (none) -> https://www.mouser.de/ProductDetail/KEMET/C1210C105K1RACAUTO
- C304: footprint Tripmaster:C_1206_3216 -> Capacitor_SMD:C_1210_3225Metric; MPN (none) -> C1210C105K1RACAUTO; Supplier_URL (none) -> https://www.mouser.de/ProductDetail/KEMET/C1210C105K1RACAUTO
- C305: MPN (none) -> C1210C104KARACAUTO; Supplier_URL (none) -> https://www.mouser.de/de/ProductDetail/KEMET/C1210C104KARAC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
Changed lines of the file:
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@@
 (symbol (lib_id "Tripmaster_Sym:R") (at 149.86 299.72 0) (unit 1) (in_bom yes) (on_board yes) (dnp no) (property "Reference" "R320" (at 149.86 285.75 0) (effects (font (size 1 1)))) (property "Value" "100R dVdt-C SERIES (TI)" (at 149.86 288.29 0) (effects (font (size 1 1)))) (property "Footprint" "Tripmaster:R_1206_3216" (at 149.86 299.72 0) (effects (font (size 1.0 1.0)) (hide yes))) (pin "1") (pin "2") (instances (project "TripPower_5V2A" (path "/f1512578-cc72-4c26-bf70-dbbd00000001/f1512578-cc72-4c26-bf70-dbbd00000002" (reference "R320") (unit 1)))))
 (symbol (lib_id "Tripmaster_Sym:C") (at 234.95 299.72 0) (unit 1) (in_bom yes) (on_board yes) (dnp no) (property "Reference" "C301" (at 234.95 285.75 0) (effects (font (size 1 1)))) (property "Value" "47nF 50V TMR" (at 234.95 288.29 0) (effects (font (size 1 1)))) (property "Footprint" "Tripmaster:C_1206_3216" (at 234.95 299.72 0) (effects (font (size 1.0 1.0)) (hide yes))) (pin "1") (pin "2") (instances (project "TripPower_5V2A" (path "/f1512578-cc72-4c26-bf70-dbbd00000001/f1512578-cc72-4c26-bf70-dbbd00000002" (reference "C301") (unit 1)))))
-(symbol (lib_id "Tripmaster_Sym:C") (at 320.04 299.72 0) (unit 1) (in_bom yes) (on_board yes) (dnp no) (property "Reference" "C302" (at 320.04 285.75 0) (effects (font (size 1 1)))) (property "Value" "1uF 100V VS CLAMP" (at 320.04 288.29 0) (effects (font (size 1 1)))) (property "Footprint" "Tripmaster:C_1210_3225" (at 320.04 299.72 0) (effects (font (size 1.0 1.0)) (hide yes))) (pin "1") (pin "2") (instances (project "TripPower_5V2A" (path "/f1512578-cc72-4c26-bf70-dbbd00000001/f1512578-cc72-4c26-bf70-dbbd00000002" (reference "C302") (unit 1)))))
+(symbol (lib_id "Tripmaster_Sym:C") (at 320.04 299.72 0) (unit 1) (in_bom yes) (on_board yes) (dnp no) (property "Reference" "C302" (at 320.04 285.75 0) (effects (font (size 1 1)))) (property "Value" "1uF 100V VS CLAMP" (at 320.04 288.29 0) (effects (font (size 1 1)))) (property "Footprint" "Tripmaster:C_1210_3225" (at 320.04 299.72 0) (effects (font (size 1.0 1.0)) (hide yes))) (property "MPN" "C1210C105K1RACAUTO" (at 0 0 0) (effects (font (size 1 1)) (hide yes))) (property "Supplier_URL" "https://www.mouser.de/ProductDetail/KEMET/C1210C105K1RACAUTO" (at 0 0 0) (effects (font (size 1 1)) (hide yes))) (pin "1") (pin "2") (instances (project "TripPower_5V2A" (path "/f1512578-cc72-4c26-bf70-dbbd00000001/f1512578-cc72-4c26-bf70-dbbd00000002" (reference "C302") (unit 1)))))
 (symbol (lib_id "Tripmaster_Sym:C") (at 405.13 299.72 0) (unit 1) (in_bom yes) (on_board yes) (dnp no) (property "Reference" "C303" (at 405.13 285.75 0) (effects (font (size 1 1)))) (property "Value" "470nF 100V X7R AEC-Q200" (at 405.13 288.29 0) (effects (font (size 1 1)))) (property "Footprint" "Capacitor_SMD:C_1206_3216Metric" (at 405.13 299.72 0) (effects (font (size 1.0 1.0)) (hide yes))) (property "MPN" "C1206C474K1RECAUTO7210" (at 0 0 0) (effects (font (size 1 1)) (hide yes))) (property "Supplier_URL" "https://www.mouser.de/de/ProductDetail/KEMET/C1206C474K1RECAUTO7210" (at 0 0 0) (effects (font (size 1 1)) (hide yes))) (property "Alternative_MPN" "CGA5L2X7R2A474K160AA" (at 0 0 0) (effects (font (size 1 1)) (hide yes))) (pin "1") (pin "2") (instances (project "TripPower_5V2A" (path "/f1512578-cc72-4c26-bf70-dbbd00000001/f1512578-cc72-4c26-bf70-dbbd00000002" (reference "C303") (unit 1)))))
-(symbol (lib_id "Tripmaster_Sym:C") (at 490.22 299.72 0) (unit 1) (in_bom yes) (on_board yes) (dnp no) (property "Reference" "C304" (at 490.22 285.75 0) (effects (font (size 1 1)))) (property "Value" "1uF 100V A BYPASS" (at 490.22 288.29 0) (effects (font (size 1 1)))) (property "Footprint" "Tripmaster:C_1206_3216" (at 490.22 299.72 0) (effects (font (size 1.0 1.0)) (hide yes))) (pin "1") (pin "2") (instances (project "TripPower_5V2A" (path "/f1512578-cc72-4c26-bf70-dbbd00000001/f1512578-cc72-4c26-bf70-dbbd00000002" (reference "C304") (unit 1)))))
-(symbol (lib_id "Tripmaster_Sym:C") (at 64.77 325.12 0) (unit 1) (in_bom yes) (on_board yes) (dnp no) (property "Reference" "C305" (at 64.77 311.15 0) (effects (font (size 1 1)))) (property "Value" "100nF 250V VIN HF" (at 64.77 313.69 0) (effects (font (size 1 1)))) (property "Footprint" "Tripmaster:C_1210_3225" (at 64.77 325.12 0) (effects (font (size 1.0 1.0)) (hide yes))) (pin "1") (pin "2") (instances (project "TripPower_5V2A" (path "/f1512578-cc72-4c26-bf70-dbbd00000001/f1512578-cc72-4c26-bf70-dbbd00000002" (reference "C305") (unit 1)))))
+(symbol (lib_id "Tripmaster_Sym:C") (at 490.22 299.72 0) (unit 1) (in_bom yes) (on_board yes) (dnp no) (property "Reference" "C304" (at 490.22 285.75 0) (effects (font (size 1 1)))) (property "Value" "1uF 100V A BYPASS" (at 490.22 288.29 0) (effects (font (size 1 1)))) (property "Footprint" "Capacitor_SMD:C_1210_3225Metric" (at 490.22 299.72 0) (effects (font (size 1.0 1.0)) (hide yes))) (property "MPN" "C1210C105K1RACAUTO" (at 0 0 0) (effects (font (size 1 1)) (hide yes))) (property "Supplier_URL" "https://www.mouser.de/ProductDetail/KEMET/C1210C105K1RACAUTO" (at 0 0 0) (effects (font (size 1 1)) (hide yes))) (pin "1") (pin "2") (instances (project "TripPower_5V2A" (path "/f1512578-cc72-4c26-bf70-dbbd00000001/f1512578-cc72-4c26-bf70-dbbd00000002" (reference "C304") (unit 1)))))
+(symbol (lib_id "Tripmaster_Sym:C") (at 64.77 325.12 0) (unit 1) (in_bom yes) (on_board yes) (dnp no) (property "Reference" "C305" (at 64.77 311.15 0) (effects (font (size 1 1)))) (property "Value" "100nF 250V VIN HF" (at 64.77 313.69 0) (effects (font (size 1 1)))) (property "Footprint" "Tripmaster:C_1210_3225" (at 64.77 325.12 0) (effects (font (size 1.0 1.0)) (hide yes))) (property "MPN" "C1210C104KARACAUTO" (at 0 0 0) (effects (font (size 1 1)) (hide yes))) (property "Supplier_URL" "https://www.mouser.de/de/ProductDetail/KEMET/C1210C104KARACAUTO" (at 0 0 0) (effects (font (size 1 1)) (hide yes))) (pin "1") (pin "2") (instances (project "TripPower_5V2A" (path "/f1512578-cc72-4c26-bf70-dbbd00000001/f1512578-cc72-4c26-bf70-dbbd00000002" (reference "C305") (unit 1)))))
 (symbol (lib_id "TripTracer_V1:PWR_CPOL") (at 149.86 325.12 0) (unit 1) (in_bom yes) (on_board yes) (dnp no) (property "Reference" "C306" (at 149.86 311.15 0) (effects (font (size 1 1)))) (property "Value" "47uF 63V POST SHUNT" (at 149.86 313.69 0) (effects (font (size 1 1)))) (property "Footprint" "Capacitor_SMD:CP_Elec_8x10.5" (at 149.86 325.12 0) (effects (font (size 1.0 1.0)) (hide yes))) (pin "1") (pin "2") (instances (project "TripPower_5V2A" (path "/f1512578-cc72-4c26-bf70-dbbd00000001/f1512578-cc72-4c26-bf70-dbbd00000002" (reference "C306") (unit 1)))))
 (symbol (lib_id "TripTracer_V1:PWR_DIODE") (at 234.95 325.12 0) (unit 1) (in_bom yes) (on_board yes) (dnp no) (property "Reference" "D301" (at 234.95 311.15 0) (effects (font (size 1 1)))) (property "Value" "1SMB5943BT3G 56V ZENER" (at 234.95 313.69 0) (effects (font (size 1 1)))) (property "Footprint" "Diode_SMD:D_SMB" (at 234.95 325.12 0) (effects (font (size 1.0 1.0)) (hide yes))) (pin "1") (pin "2") (instances (project "TripPower_5V2A" (path "/f1512578-cc72-4c26-bf70-dbbd00000001/f1512578-cc72-4c26-bf70-dbbd00000002" (reference "D301") (unit 1)))))

Commit message: fix(TripPower): lock 2W 5mOhm shunt and AEC-Q200 750k OV/UV divider resistor MPNs
Parts:
- R301: MPN (none) -> RLM25FEER005; Supplier_URL (none) -> https://www.lcsc.com/product-detail/C185817.html
- R307, R308, R310, R311: MPN (none) -> AC1206FR-07750KL; Supplier_URL (none) -> https://yageogroup.com/component-documentation/download/spe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

Commit message: bom(TripPower): reflect verified 2W current shunt rating on KiCad value
Parts:
- R301: value 5mR 1% 2512 >=1W -> 5mR 1% 2512 2W TA-I
Changed lines of the file:
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@@
 (symbol (lib_id "TripPower_Sym:TripleTerminal") (at 66.04 157.48 0) (unit 1) (in_bom yes) (on_board yes) (dnp no) (property "Reference" "J301" (at 66.04 143.51 0) (effects (font (size 1 1)))) (property "Value" "INPUT: VIN/RUN/GND" (at 66.04 146.05 0) (effects (font (size 1 1)))) (property "Footprint" "Tripmaster:Vehicle_Pigtail_3Wire" (at 66.04 157.48 0) (effects (font (size 1.0 1.0)) (hide yes))) (pin "1") (pin "2") (pin "3") (instances (project "TripPower_5V2A" (path "/f1512578-cc72-4c26-bf70-dbbd00000001/f1512578-cc72-4c26-bf70-dbbd00000002" (reference "J301") (unit 1)))))
 (symbol (lib_id "TripPower_Sym:TripleTerminal") (at 472.44 157.48 0) (unit 1) (in_bom yes) (on_board yes) (dnp no) (property "Reference" "J302" (at 472.44 143.51 0) (effects (font (size 1 1)))) (property "Value" "OUT: PROT_UNFUSED/5V/GND" (at 472.44 146.05 0) (effects (font (size 1 1)))) (property "Footprint" "Tripmaster:Vehicle_Pigtail_3Wire" (at 472.44 157.48 0) (effects (font (size 1.0 1.0)) (hide yes))) (pin "1") (pin "2") (pin "3") (instances (project "TripPower_5V2A" (path "/f1512578-cc72-4c26-bf70-dbbd00000001/f1512578-cc72-4c26-bf70-dbbd00000002" (reference "J302") (unit 1)))))
-(symbol (lib_id "Tripmaster_Sym:R") (at 64.77 224.79 0) (unit 1) (in_bom yes) (on_board yes) (dnp no) (property "Reference" "R301" (at 64.77 210.82 0) (effects (font (size 1 1)))) (property "Value" "5mR 1% 2512 >=1W" (at 64.77 213.36 0) (effects (font (size 1 1)))) (property "Footprint" "Resistor_SMD:R_2512_6332Metric" (at 64.77 224.79 0) (effects (font (size 1.0 1.0)) (hide yes))) (property "MPN" "RLM25FEER005" (at 0 0 0) (effects (font (size 1 1)) (hide yes))) (property "Supplier_URL" "https://www.lcsc.com/product-detail/C185817.html" (at 0 0 0) (effects (font (size 1 1)) (hide yes))) (pin "1") (pin "2") (instances (project "TripPower_5V2A" (path "/f1512578-cc72-4c26-bf70-dbbd00000001/f1512578-cc72-4c26-bf70-dbbd00000002" (reference "R301") (unit 1)))))
+(symbol (lib_id "Tripmaster_Sym:R") (at 64.77 224.79 0) (unit 1) (in_bom yes) (on_board yes) (dnp no) (property "Reference" "R301" (at 64.77 210.82 0) (effects (font (size 1 1)))) (property "Value" "5mR 1% 2512 2W TA-I" (at 64.77 213.36 0) (effects (font (size 1 1)))) (property "Footprint" "Resistor_SMD:R_2512_6332Metric" (at 64.77 224.79 0) (effects (font (size 1.0 1.0)) (hide yes))) (property "MPN" "RLM25FEER005" (at 0 0 0) (effects (font (size 1 1)) (hide yes))) (property "Supplier_URL" "https://www.lcsc.com/product-detail/C185817.html" (at 0 0 0) (effects (font (size 1 1)) (hide yes))) (pin "1") (pin "2") (instances (project "TripPower_5V2A" (path "/f1512578-cc72-4c26-bf70-dbbd00000001/f1512578-cc72-4c26-bf70-dbbd00000002" (reference "R301") (unit 1)))))
 (symbol (lib_id "Tripmaster_Sym:R") (at 149.86 224.79 0) (unit 1) (in_bom yes) (on_board yes) (dnp no) (property "Reference" "R302" (at 149.86 210.82 0) (effects (font (size 1 1)))) (property "Value" "50R RSET" (at 149.86 213.36 0) (effects (font (size 1 1)))) (property "Footprint" "Tripmaster:R_1206_3216" (at 149.86 224.79 0) (effects (font (size 1.0 1.0)) (hide yes))) (pin "1") (pin "2") (instances (project "TripPower_5V2A" (path "/f1512578-cc72-4c26-bf70-dbbd00000001/f1512578-cc72-4c26-bf70-dbbd00000002" (reference "R302") (unit 1)))))
 (symbol (lib_id "Tripmaster_Sym:R") (at 234.95 224.79 0) (unit 1) (in_bom yes) (on_board yes) (dnp no) (property "Reference" "R303" (at 234.95 210.82 0) (effects (font (size 1 1)))) (property "Value" "470R RISCP" (at 234.95 213.36 0) (effects (font (size 1 1)))) (property "Footprint" "Tripmaster:R_1206_3216" (at 234.95 224.79 0) (effects (font (size 1.0 1.0)) (hide yes))) (pin "1") (pin "2") (instances (project "TripPower_5V2A" (path "/f1512578-cc72-4c26-bf70-dbbd00000001/f1512578-cc72-4c26-bf70-dbbd00000002" (reference "R303") (unit 1)))))
