File: hardware/modules/TripPower_5V2A/01_Protection_LM74930.kicad_sch (KiCad schematic)
At the start: 41 parts, among them J301 INPUT: VIN/RUN/GND, J302 OUT: PROT_UNFUSED/5V/GND, Q301 SQM10250E_GE3 250V CANDIDATE, Q302 BUK7Y4R8-60EX 60V CANDIDATE, U301 LM74930QRGERQ1

Commit message: refactor(TripPower REV5): remove obsolete EN BJT output R316/R318, BAS116 D305 and legacy C309 including orphan labels
Parts:
- removed C309: 10uF 50V EN DELAY WIP, Capacitor_SMD:C_1210_3225Metric, symbol Tripmaster_Sym:C
- removed D305: REV5 DNP LEGACY D305, Package_TO_SOT_SMD:SOT-23, symbol TripPower_Sym:BAS116Q_A1_K3_NC2
- removed R316: REV5 DNP LEGACY R316, Tripmaster:R_1206_3216, symbol Tripmaster_Sym:R
- removed R318: REV5 DNP LEGACY R318, Tripmaster:R_1206_3216, symbol Tripmaster_Sym:R
Changed lines of the file:
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@@
 (symbol (lib_id "Tripmaster_Sym:R") (at 149.86 275.59 0) (unit 1) (in_bom yes) (on_board yes) (dnp no) (property "Reference" "R314" (at 149.86 261.62 0) (effects (font (size 1 1)))) (property "Value" "3.3k 2512 PULSE CANDIDATE" (at 149.86 264.16 0) (effects (font (size 1 1)))) (property "Footprint" "Resistor_SMD:R_2512_6332Metric" (at 149.86 275.59 0) (effects (font (size 1.0 1.0)) (hide yes))) (property "MPN" "CRCW25123K30FKEGHP" (at 0 0 0) (effects (font (size 1 1)) (hide yes))) (pin "1") (pin "2") (instances (project "TripPower_5V2A" (path "/f1512578-cc72-4c26-bf70-dbbd00000001/f1512578-cc72-4c26-bf70-dbbd00000002" (reference "R314") (unit 1)))))
 (symbol (lib_id "Tripmaster_Sym:R") (at 234.95 275.59 0) (unit 1) (in_bom yes) (on_board yes) (dnp no) (property "Reference" "R315" (at 234.95 261.62 0) (effects (font (size 1 1)))) (property "Value" "3.3k 2512 PULSE CANDIDATE" (at 234.95 264.16 0) (effects (font (size 1 1)))) (property "Footprint" "Resistor_SMD:R_2512_6332Metric" (at 234.95 275.59 0) (effects (font (size 1.0 1.0)) (hide yes))) (property "MPN" "CRCW25123K30FKEGHP" (at 0 0 0) (effects (font (size 1 1)) (hide yes))) (pin "1") (pin "2") (instances (project "TripPower_5V2A" (path "/f1512578-cc72-4c26-bf70-dbbd00000001/f1512578-cc72-4c26-bf70-dbbd00000002" (reference "R315") (unit 1)))))
-(symbol (lib_id "Tripmaster_Sym:R") (at 320.04 275.59 0) (unit 1) (in_bom yes) (on_board yes) (dnp yes) (property "Reference" "R316" (at 320.04 261.62 0) (effects (font (size 1 1)))) (property "Value" "REV5 DNP LEGACY R316" (at 320.04 264.16 0) (effects (font (size 1 1)))) (property "Footprint" "Tripmaster:R_1206_3216" (at 320.04 275.59 0) (effects (font (size 1.0 1.0)) (hide yes))) (pin "1") (pin "2") (instances (project "TripPower_5V2A" (path "/f1512578-cc72-4c26-bf70-dbbd00000001/f1512578-cc72-4c26-bf70-dbbd00000002" (reference "R316") (unit 1)))))
 (symbol (lib_id "Tripmaster_Sym:R") (at 405.13 275.59 0) (unit 1) (in_bom yes) (on_board yes) (dnp yes) (property "Reference" "R317" (at 405.13 261.62 0) (effects (font (size 1 1)))) (property "Value" "1M 1% RUN_CMD TO SENSE2 - RUN ONLY" (at 405.13 264.16 0) (effects (font (size 1 1)))) (property "Footprint" "Tripmaster:R_1206_3216" (at 405.13 275.59 0) (effects (font (size 1.0 1.0)) (hide yes))) (property "MPN" "RC1206FR-071ML" (at 0 0 0) (effects (font (size 1 1)) (hide yes))) (pin "1") (pin "2") (instances (project "TripPower_5V2A" (path "/f1512578-cc72-4c26-bf70-dbbd00000001/f1512578-cc72-4c26-bf70-dbbd00000002" (reference "R317") (unit 1)))))
-(symbol (lib_id "Tripmaster_Sym:R") (at 490.22 275.59 0) (unit 1) (in_bom yes) (on_board yes) (dnp yes) (property "Reference" "R318" (at 490.22 261.62 0) (effects (font (size 1 1)))) (property "Value" "REV5 DNP LEGACY R318" (at 490.22 264.16 0) (effects (font (size 1 1)))) (property "Footprint" "Tripmaster:R_1206_3216" (at 490.22 275.59 0) (effects (font (size 1.0 1.0)) (hide yes))) (pin "1") (pin "2") (instances (project "TripPower_5V2A" (path "/f1512578-cc72-4c26-bf70-dbbd00000001/f1512578-cc72-4c26-bf70-dbbd00000002" (reference "R318") (unit 1)))))
 (symbol (lib_id "Tripmaster_Sym:R") (at 64.77 299.72 0) (unit 1) (in_bom yes) (on_board yes) (dnp no) (property "Reference" "R319" (at 64.77 285.75 0) (effects (font (size 1 1)))) (property "Value" "0R AUTO VS TO RUN_SENSE; DNP IN RUN" (at 64.77 288.29 0) (effects (font (size 1 1)))) (property "Footprint" "Tripmaster:R_1206_3216" (at 64.77 299.72 0) (effects (font (size 1.0 1.0)) (hide yes))) (property "MPN" "RC1206JR-070RL" (at 0 0 0) (effects (font (size 1 1)) (hide yes))) (pin "1") (pin "2") (instances (project "TripPower_5V2A" (path "/f1512578-cc72-4c26-bf70-dbbd00000001/f1512578-cc72-4c26-bf70-dbbd00000002" (reference "R319") (unit 1)))))
 (symbol (lib_id "Tripmaster_Sym:R") (at 149.86 299.72 0) (unit 1) (in_bom yes) (on_board yes) (dnp no) (property "Reference" "R320" (at 149.86 285.75 0) (effects (font (size 1 1)))) (property "Value" "100R dVdt-C SERIES (TI)" (at 149.86 288.29 0) (effects (font (size 1 1)))) (property "Footprint" "Tripmaster:R_1206_3216" (at 149.86 299.72 0) (effects (font (size 1.0 1.0)) (hide yes))) (pin "1") (pin "2") (instances (project "TripPower_5V2A" (path "/f1512578-cc72-4c26-bf70-dbbd00000001/f1512578-cc72-4c26-bf70-dbbd00000002" (reference "R320") (unit 1)))))
@@
 (wire (pts (xy 246.38 275.59) (xy 251.46 275.59)) (stroke (width 0) (type default)))
 (global_label "VS_CLAMP" (shape bidirectional) (at 251.46 275.59 0) (effects (font (size 0.9 0.9)) (justify left)))
-(wire (pts (xy 308.61 275.59) (xy 303.53 275.59)) (stroke (width 0) (type default)))
-(global_label "CTRL_EN" (shape bidirectional) (at 303.53 275.59 0) (effects (font (size 0.9 0.9)) (justify left)))
-(wire (pts (xy 331.47 275.59) (xy 336.55 275.59)) (stroke (width 0) (type default)))
-(global_label "GND" (shape bidirectional) (at 336.55 275.59 0) (effects (font (size 0.9 0.9)) (justify left)))
 (wire (pts (xy 393.7 275.59) (xy 388.62 275.59)) (stroke (width 0) (type default)))
 (global_label "RUN_CMD" (shape bidirectional) (at 388.62 275.59 0) (effects (font (size 0.9 0.9)) (justify left)))
 (wire (pts (xy 416.56 275.59) (xy 421.64 275.59)) (stroke (width 0) (type default)))
 (global_label "RUN_SENSE" (shape bidirectional) (at 421.64 275.59 0) (effects (font (size 0.9 0.9)) (justify left)))
-(wire (pts (xy 478.79 275.59) (xy 473.71 275.59)) (stroke (width 0) (type default)))
-(global_label "PNP_OUT" (shape bidirectional) (at 473.71 275.59 0) (effects (font (size 0.9 0.9)) (justify left)))
-(wire (pts (xy 501.65 275.59) (xy 506.73 275.59)) (stroke (width 0) (type default)))
-(global_label "CTRL_EN" (shape bidirectional) (at 506.73 275.59 0) (effects (font (size 0.9 0.9)) (justify left)))
 (wire (pts (xy 53.34 299.72) (xy 48.26 299.72)) (stroke (width 0) (type default)))
 (global_label "VS_CLAMP" (shape bidirectional) (at 48.26 299.72 0) (effects (font (size 0.9 0.9)) (justify left)))
@@
 (global_label "FAULT_OC_N" (shape bidirectional) (at 48.26 400.05 0) (effects (font (size 0.9 0.9)) (justify left)))
 (global_label "5V_OUT" (shape bidirectional) (at 81.28 400.05 0) (effects (font (size 0.9 0.9)) (justify left)))
-(symbol (lib_id "TripPower_Sym:BAS116Q_A1_K3_NC2") (at 151.13 400.05 0) (unit 1) (in_bom yes) (on_board yes) (dnp yes)
-(property "Reference" "D305" (at 151.13 384.81 0) (effects (font (size 1 1))))
-(property "Value" "REV5 DNP LEGACY D305" (at 151.13 388.62 0) (effects (font (size 1 1))))
-(property "Footprint" "Package_TO_SOT_SMD:SOT-23" (at 151.13 400.05 0) (effects (font (size 1 1)) (hide yes)))
-(pin "1") (pin "3") (pin "2")
-(instances (project "TripPower_5V2A" (path "/f1512578-cc72-4c26-bf70-dbbd00000001/f1512578-cc72-4c26-bf70-dbbd00000002" (reference "D305") (unit 1)))))
-(wire (pts (xy 140.97 400.05) (xy 135.89 400.05)) (stroke (width 0) (type default)))
-(global_label "RUN_SINK_C" (shape bidirectional) (at 135.89 400.05 0) (effects (font (size 0.9 0.9)) (justify left)))
-(wire (pts (xy 161.29 400.05) (xy 166.37 400.05)) (stroke (width 0) (type default)))
-(global_label "RUN_BYPASS_NODE" (shape bidirectional) (at 166.37 400.05 0) (effects (font (size 0.9 0.9)) (justify left)))
 (symbol (lib_id "Tripmaster_Sym:C") (at 149.86 350.52 0) (unit 1) (in_bom yes) (on_board yes) (dnp no) (property "Reference" "C307" (at 149.86 336.55 0) (effects (font (size 1 1)))) (property "Value" "10nF 250V dVdt WIP" (at 149.86 339.09 0) (effects (font (size 1 1)))) (property "Footprint" "Tripmaster:C_1206_3216" (at 149.86 350.52 0) (effects (font (size 1.0 1.0)) (hide yes))) (property "MPN" "C1206C103JARECAUTO" (at 0 0 0) (effects (font (size 1 1)) (hide yes))) (property "Datasheet" "https://www.digikey.de/en/products/detail/kemet/C1206C103JARECAUTO/16680107" (at 0 0 0) (effects (font (size 1 1)) (hide yes))) (pin "1") (pin "2") (instances (project "TripPower_5V2A" (path "/f1512578-cc72-4c26-bf70-dbbd00000001/f1512578-cc72-4c26-bf70-dbbd00000002" (reference "C307") (unit 1)))))
 (wire (pts (xy 138.43 350.52) (xy 133.35 350.52)) (stroke (width 0) (type default)))
@@
 (wire (pts (xy 501.65 350.52) (xy 506.73 350.52)) (stroke (width 0) (type default)))
 (global_label "GND" (shape bidirectional) (at 506.73 350.52 0) (effects (font (size 0.9 0.9)) (justify left)))
-(symbol (lib_id "Tripmaster_Sym:C") (at 405.13 350.52 0) (unit 1) (in_bom yes) (on_board yes) (dnp yes) (property "Reference" "C309" (at 405.13 336.55 0) (effects (font (size 1 1)))) (property "Value" "10uF 50V EN DELAY WIP" (at 405.13 339.09 0) (effects (font (size 1 1)))) (property "Footprint" "Capacitor_SMD:C_1210_3225Metric" (at 405.13 350.52 0) (effects (font (size 1.0 1.0)) (hide yes))) (property "MPN" "12105C106K4T2A" (at 0 0 0) (effects (font (size 1 1)) (hide yes))) (property "Supplier_URL" "https://www.mouser.de/de/ProductDetail/KEMET/12105C106K4T2A" (at 0 0 0) (effects (font (size 1 1)) (hide yes))) (property "Status" "DNP; supervisor U302 controls Q303 series enable, no RC delay" (at 0 0 0) (effects (font (size 1 1)) (hide yes))) (pin "1") (pin "2") (instances (project "TripPower_5V2A" (path "/f1512578-cc72-4c26-bf70-dbbd00000001/f1512578-cc72-4c26-bf70-dbbd00000002" (reference "C309") (unit 1)))))
-(wire (pts (xy 393.7 350.52) (xy 388.62 350.52)) (stroke (width 0) (type default)))
-(global_label "CTRL_EN" (shape bidirectional) (at 388.62 350.52 0) (effects (font (size 0.9 0.9)) (justify left)))
-(wire (pts (xy 416.56 350.52) (xy 421.64 350.52)) (stroke (width 0) (type default)))
-(global_label "GND" (shape bidirectional) (at 421.64 350.52 0) (effects (font (size 0.9 0.9)) (justify left)))
  (embedded_fonts no))

Commit message: TripPower REV5: DNP unused IMON load and FLT pullup
Parts:
- R305, R321: now not fitted
Changed lines of the file:
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@@
 (symbol (lib_id "Tripmaster_Sym:R") (at 234.95 224.79 0) (unit 1) (in_bom yes) (on_board yes) (dnp no) (property "Reference" "R303" (at 234.95 210.82 0) (effects (font (size 1 1)))) (property "Value" "470R RISCP" (at 234.95 213.36 0) (effects (font (size 1 1)))) (property "Footprint" "Tripmaster:R_1206_3216" (at 234.95 224.79 0) (effects (font (size 1.0 1.0)) (hide yes))) (pin "1") (pin "2") (instances (project "TripPower_5V2A" (path "/f1512578-cc72-4c26-bf70-dbbd00000001/f1512578-cc72-4c26-bf70-dbbd00000002" (reference "R303") (unit 1)))))
 (symbol (lib_id "Tripmaster_Sym:R") (at 320.04 224.79 0) (unit 1) (in_bom yes) (on_board yes) (dnp no) (property "Reference" "R304" (at 320.04 210.82 0) (effects (font (size 1 1)))) (property "Value" "33.2k RILIM" (at 320.04 213.36 0) (effects (font (size 1 1)))) (property "Footprint" "Tripmaster:R_1206_3216" (at 320.04 224.79 0) (effects (font (size 1.0 1.0)) (hide yes))) (pin "1") (pin "2") (instances (project "TripPower_5V2A" (path "/f1512578-cc72-4c26-bf70-dbbd00000001/f1512578-cc72-4c26-bf70-dbbd00000002" (reference "R304") (unit 1)))))
-(symbol (lib_id "Tripmaster_Sym:R") (at 405.13 224.79 0) (unit 1) (in_bom yes) (on_board yes) (dnp no) (property "Reference" "R305" (at 405.13 210.82 0) (effects (font (size 1 1)))) (property "Value" "6.8k RIMON" (at 405.13 213.36 0) (effects (font (size 1 1)))) (property "Footprint" "Tripmaster:R_1206_3216" (at 405.13 224.79 0) (effects (font (size 1.0 1.0)) (hide yes))) (pin "1") (pin "2") (instances (project "TripPower_5V2A" (path "/f1512578-cc72-4c26-bf70-dbbd00000001/f1512578-cc72-4c26-bf70-dbbd00000002" (reference "R305") (unit 1)))))
+(symbol (lib_id "Tripmaster_Sym:R") (at 405.13 224.79 0) (unit 1) (in_bom yes) (on_board yes) (dnp yes) (property "Reference" "R305" (at 405.13 210.82 0) (effects (font (size 1 1)))) (property "Value" "6.8k RIMON" (at 405.13 213.36 0) (effects (font (size 1 1)))) (property "Footprint" "Tripmaster:R_1206_3216" (at 405.13 224.79 0) (effects (font (size 1.0 1.0)) (hide yes))) (pin "1") (pin "2") (instances (project "TripPower_5V2A" (path "/f1512578-cc72-4c26-bf70-dbbd00000001/f1512578-cc72-4c26-bf70-dbbd00000002" (reference "R305") (unit 1)))))
 (symbol (lib_id "Tripmaster_Sym:R") (at 490.22 224.79 0) (unit 1) (in_bom yes) (on_board yes) (dnp no) (property "Reference" "R306" (at 490.22 210.82 0) (effects (font (size 1 1)))) (property "Value" "100k RTMR LATCH" (at 490.22 213.36 0) (effects (font (size 1 1)))) (property "Footprint" "Tripmaster:R_1206_3216" (at 490.22 224.79 0) (effects (font (size 1.0 1.0)) (hide yes))) (pin "1") (pin "2") (instances (project "TripPower_5V2A" (path "/f1512578-cc72-4c26-bf70-dbbd00000001/f1512578-cc72-4c26-bf70-dbbd00000002" (reference "R306") (unit 1)))))
 (symbol (lib_id "Tripmaster_Sym:R") (at 64.77 250.19 0) (unit 1) (in_bom yes) (on_board yes) (dnp no) (property "Reference" "R307" (at 64.77 236.22 0) (effects (font (size 1 1)))) (property "Value" "750k 1% OV HIGH 1" (at 64.77 238.76 0) (effects (font (size 1 1)))) (property "Footprint" "Tripmaster:R_1206_3216" (at 64.77 250.19 0) (effects (font (size 1.0 1.0)) (hide yes))) (property "MPN" "AC1206FR-07750KL" (at 0 0 0) (effects (font (size 1 1)) (hide yes))) (property "Supplier_URL" "https://yageogroup.com/component-documentation/download/specsheet/AC1206FR-07750KL" (at 0 0 0) (effects (font (size 1 1)) (hide yes))) (pin "1") (pin "2") (instances (project "TripPower_5V2A" (path "/f1512578-cc72-4c26-bf70-dbbd00000001/f1512578-cc72-4c26-bf70-dbbd00000002" (reference "R307") (unit 1)))))
@@
 (instances (project "TripPower_5V2A" (path "/f1512578-cc72-4c26-bf70-dbbd00000001/f1512578-cc72-4c26-bf70-dbbd00000002" (reference "#FLG304") (unit 1)))))
 (global_label "VIN_PROTECTED_UNFUSED" (shape bidirectional) (at 38.1 104.14 0) (effects (font (size 1 1)) (justify left)))
-(symbol (lib_id "Tripmaster_Sym:R") (at 64.77 400.05 0) (unit 1) (in_bom yes) (on_board yes) (dnp no)
+(symbol (lib_id "Tripmaster_Sym:R") (at 64.77 400.05 0) (unit 1) (in_bom yes) (on_board yes) (dnp yes)
  (property "Reference" "R321" (at 64.77 386.08 0) (effects (font (size 1 1))))
  (property "Value" "47k 1% FLT TO 5V" (at 64.77 388.62 0) (effects (font (size 1 1))))
