File: hardware/modules/TripPower_5V2A/03_VS_READY_TPS3760.kicad_sch (KiCad schematic)
At the start: 7 parts, among them U302 TPS3760A012DYYRQ1

Commit message: feat(TripPower): implement RESET-qualified AUTO/RUN series EN interlock with automotive MOSFET, clamps and C309 DNP
Parts:
- added D306: BAS70-02V-HG3-08 GATE TO RESET SCHOTTKY, Diode_SMD:D_SOD-523, symbol TripTracer_V1:PWR_DIODE
- added D307: SZMMSZ5240BT1G 10V GATE ZENER, Diode_SMD:D_SOD-123, symbol TripTracer_V1:PWR_DIODE
- added D308: BAS70-02V-HG3-08 EN FAILSAFE CLAMP, Diode_SMD:D_SOD-523, symbol TripTracer_V1:PWR_DIODE
- added Q303: BVSS123LT1G 100V AEC-Q101, Package_TO_SOT_SMD:SOT-23, symbol TripPower_Sym:EN_PASS_NMOS_GSD
- added R334: 470k 1% VS GATE DRIVE, Resistor_SMD:R_1206_3216Metric, symbol Tripmaster_Sym:R
- added R335: 1M 1% GATE PULLDOWN, Resistor_SMD:R_1206_3216Metric, symbol Tripmaster_Sym:R
Connections:
- net GND: now also D307.2 (A), R335.2
- net VS_CLAMP: now also R334.1
- net VS_READY_RESET_OD_PRELIM: now also D306.1 (K), D308.1 (K)
- new net CTRL_EN: D308.2 (A), Q303.2 (S)
- new net EN_GATE_DRIVE: D306.2 (A), D307.1 (K), Q303.1 (G), R334.2, R335.1
- new net EN_REQUEST_RAW: Q303.3 (D)
Other:
- note added: "Q303 series EN pass: AUTO R319 and RUN D305 feed EN_REQUEST_RAW (NO bypass); RESET asserted LOW drives D306 gate clamp and D308 EN clamp. Gate VS divider R334/R335; D307 10V gate Zener. C309 DNP. All cold/hot/leakage/surge gates OPEN."
- note removed: "NOT CONNECTED TO CTRL_EN YET: complete guaranteed fail-safe AUTO/RUN AND interlock first. U302 TPS3760 automotive chosen; 8.07V rise / 6.04V fall nominal resistor model ONLY, 250ms CTR delay only approximate. C309 remains experimental."
- title: TripPower VS_READY adjustable supervisor; output NOT WIRED TO CTRL_EN -> TripPower VS_READY adjustable supervisor; AUTO/RUN via gated Q303 to CTRL_EN – prototype, not qualified
Changed lines of the file:
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@@
 (kicad_sch (version 20250114) (generator "eeschema")
-(paper "A4")
-(title_block (title "TripPower VS_READY adjustable supervisor; output NOT WIRED TO CTRL_EN") (date "2026-10-15") (rev "RESEARCH BLOCKER / NOT RELEASED"))
-(text "NOT CONNECTED TO CTRL_EN YET: complete guaranteed fail-safe AUTO/RUN AND interlock first. U302 TPS3760 automotive chosen; 8.07V rise / 6.04V fall nominal resistor model ONLY, 250ms CTR delay only approximate. C309 remains experimental." (at 17.78 19.05 0) (effects (font (size 1.05 1.05))))
+(paper "A3")
+(title_block (title "TripPower VS_READY adjustable supervisor; AUTO/RUN via gated Q303 to CTRL_EN – prototype, not qualified") (date "2026-10-15") (rev "RESEARCH BLOCKER / NOT RELEASED"))
+(text "Q303 series EN pass: AUTO R319 and RUN D305 feed EN_REQUEST_RAW (NO bypass); RESET asserted LOW drives D306 gate clamp and D308 EN clamp. Gate VS divider R334/R335; D307 10V gate Zener. C309 DNP. All cold/hot/leakage/surge gates OPEN." (at 17.78 19.05 0) (effects (font (size 1.05 1.05))))
 (symbol (lib_id "TripTracer_V1:TPS3760A012DYYRQ1") (at 129.54 80.01 0) (unit 1) (in_bom yes) (on_board yes) (dnp no)
 (property "Reference" "U302" (at 129.54 44.45 0) (effects (font (size 1 1))))
@@
 (wire (pts (xy 177.8 185.42) (xy 182.88 185.42)) (stroke (width 0) (type default)))
 (global_label "GND" (shape bidirectional) (at 182.88 185.42 0) (effects (font (size 0.9 0.9)) (justify left)))
+(symbol (lib_id "TripPower_Sym:EN_PASS_NMOS_GSD") (at 304.8 152.4 0) (unit 1) (in_bom yes) (on_board yes) (dnp no)
+(property "Reference" "Q303" (at 304.8 135.89000000000001 0) (effects (font (size 1 1))))
+(property "Value" "BVSS123LT1G 100V AEC-Q101" (at 304.8 138.43 0) (effects (font (size 1 1))))
+(property "Footprint" "Package_TO_SOT_SMD:SOT-23" (at 304.8 152.4 0) (effects (font (size 1 1)) (hide yes)))
+(property "MPN" "BVSS123LT1G" (at 0 0 0) (effects (font (size 1 1)) (hide yes)))
+(property "Status" "EN request pass; 202V/350ms hot SOA WIP" (at 0 0 0) (effects (font (size 1 1)) (hide yes)))
+(pin "1")
+(pin "2")
+(pin "3")
+(instances (project "TripPower_5V2A" (path "/f1512578-cc72-4c26-bf70-dbbd00000001/f1512578-cc72-4c26-bf70-dbbd00000005" (reference "Q303") (unit 1)))))
+(wire (pts (xy 289.56 152.4) (xy 284.48 152.4)) (stroke (width 0) (type default)))
+(global_label "EN_GATE_DRIVE" (shape bidirectional) (at 284.48 152.4 0) (effects (font (size 0.9 0.9)) (justify left)))
+(wire (pts (xy 320.04 147.32) (xy 325.12 147.32)) (stroke (width 0) (type default)))
+(global_label "EN_REQUEST_RAW" (shape bidirectional) (at 325.12 147.32 0) (effects (font (size 0.9 0.9)) (justify left)))
+(wire (pts (xy 320.04 157.48) (xy 325.12 157.48)) (stroke (width 0) (type default)))
+(global_label "CTRL_EN" (shape bidirectional) (at 325.12 157.48 0) (effects (font (size 0.9 0.9)) (justify left)))
+(symbol (lib_id "Tripmaster_Sym:R") (at 256.54 200.66 0) (unit 1) (in_bom yes) (on_board yes) (dnp no)
+(property "Reference" "R334" (at 256.54 184.15 0) (effects (font (size 1 1))))
+(property "Value" "470k 1% VS GATE DRIVE" (at 256.54 186.69 0) (effects (font (size 1 1))))
+(property "Footprint" "Resistor_SMD:R_1206_3216Metric" (at 256.54 200.66 0) (effects (font (size 1 1)) (hide yes)))
+(property "MPN" "MPN_TBD" (at 0 0 0) (effects (font (size 1 1)) (hide yes)))
+(pin "1")
+(pin "2")
+(instances (project "TripPower_5V2A" (path "/f1512578-cc72-4c26-bf70-dbbd00000001/f1512578-cc72-4c26-bf70-dbbd00000005" (reference "R334") (unit 1)))))
+(wire (pts (xy 245.11 200.66) (xy 240.03000000000003 200.66)) (stroke (width 0) (type default)))
+(global_label "VS_CLAMP" (shape bidirectional) (at 240.03000000000003 200.66 0) (effects (font (size 0.9 0.9)) (justify left)))
+(wire (pts (xy 267.97 200.66) (xy 273.05 200.66)) (stroke (width 0) (type default)))
+(global_label "EN_GATE_DRIVE" (shape bidirectional) (at 273.05 200.66 0) (effects (font (size 0.9 0.9)) (justify left)))
+(symbol (lib_id "Tripmaster_Sym:R") (at 345.44 200.66 0) (unit 1) (in_bom yes) (on_board yes) (dnp no)
+(property "Reference" "R335" (at 345.44 184.15 0) (effects (font (size 1 1))))
+(property "Value" "1M 1% GATE PULLDOWN" (at 345.44 186.69 0) (effects (font (size 1 1))))
+(property "Footprint" "Resistor_SMD:R_1206_3216Metric" (at 345.44 200.66 0) (effects (font (size 1 1)) (hide yes)))
+(property "MPN" "MPN_TBD" (at 0 0 0) (effects (font (size 1 1)) (hide yes)))
+(pin "1")
+(pin "2")
+(instances (project "TripPower_5V2A" (path "/f1512578-cc72-4c26-bf70-dbbd00000001/f1512578-cc72-4c26-bf70-dbbd00000005" (reference "R335") (unit 1)))))
+(wire (pts (xy 334.01 200.66) (xy 328.93 200.66)) (stroke (width 0) (type default)))
+(global_label "EN_GATE_DRIVE" (shape bidirectional) (at 328.93 200.66 0) (effects (font (size 0.9 0.9)) (justify left)))
+(wire (pts (xy 356.87 200.66) (xy 361.95 200.66)) (stroke (width 0) (type default)))
+(global_label "GND" (shape bidirectional) (at 361.95 200.66 0) (effects (font (size 0.9 0.9)) (justify left)))
+(symbol (lib_id "TripTracer_V1:PWR_DIODE") (at 256.54 236.22 0) (unit 1) (in_bom yes) (on_board yes) (dnp no)
+(property "Reference" "D306" (at 256.54 219.71 0) (effects (font (size 1 1))))
+(property "Value" "BAS70-02V-HG3-08 GATE TO RESET SCHOTTKY" (at 256.54 222.25 0) (effects (font (size 1 1))))
+(property "Footprint" "Diode_SMD:D_SOD-523" (at 256.54 236.22 0) (effects (font (size 1 1)) (hide yes)))
+(property "MPN" "BAS70-02V-HG3-08" (at 0 0 0) (effects (font (size 1 1)) (hide yes)))
+(property "K_net" "VS_READY_RESET_OD_PRELIM" (at 0 0 0) (effects (font (size 1 1)) (hide yes)))
+(property "A_net" "EN_GATE_DRIVE" (at 0 0 0) (effects (font (size 1 1)) (hide yes)))
+(pin "1")
+(pin "2")
+(instances (project "TripPower_5V2A" (path "/f1512578-cc72-4c26-bf70-dbbd00000001/f1512578-cc72-4c26-bf70-dbbd00000005" (reference "D306") (unit 1)))))
+(wire (pts (xy 246.38000000000002 236.22) (xy 241.3 236.22)) (stroke (width 0) (type default)))
+(global_label "VS_READY_RESET_OD_PRELIM" (shape bidirectional) (at 241.3 236.22 0) (effects (font (size 0.9 0.9)) (justify left)))
+(wire (pts (xy 266.70000000000005 236.22) (xy 271.78000000000003 236.22)) (stroke (width 0) (type default)))
+(global_label "EN_GATE_DRIVE" (shape bidirectional) (at 271.78000000000003 236.22 0) (effects (font (size 0.9 0.9)) (justify left)))
+(symbol (lib_id "TripTracer_V1:PWR_DIODE") (at 345.44 236.22 0) (unit 1) (in_bom yes) (on_board yes) (dnp no)
+(property "Reference" "D307" (at 345.44 219.71 0) (effects (font (size 1 1))))
+(property "Value" "SZMMSZ5240BT1G 10V GATE ZENER" (at 345.44 222.25 0) (effects (font (size 1 1))))
+(property "Footprint" "Diode_SMD:D_SOD-123" (at 345.44 236.22 0) (effects (font (size 1 1)) (hide yes)))
+(property "MPN" "SZMMSZ5240BT1G" (at 0 0 0) (effects (font (size 1 1)) (hide yes)))
+(property "K_net" "EN_GATE_DRIVE" (at 0 0 0) (effects (font (size 1 1)) (hide yes)))
+(property "A_net" "GND" (at 0 0 0) (effects (font (size 1 1)) (hide yes)))
+(pin "1")
+(pin "2")
+(instances (project "TripPower_5V2A" (path "/f1512578-cc72-4c26-bf70-dbbd00000001/f1512578-cc72-4c26-bf70-dbbd00000005" (reference "D307") (unit 1)))))
+(wire (pts (xy 335.28 236.22) (xy 330.2 236.22)) (stroke (width 0) (type default)))
+(global_label "EN_GATE_DRIVE" (shape bidirectional) (at 330.2 236.22 0) (effects (font (size 0.9 0.9)) (justify left)))
+(wire (pts (xy 355.6 236.22) (xy 360.68 236.22)) (stroke (width 0) (type default)))
+(global_label "GND" (shape bidirectional) (at 360.68 236.22 0) (effects (font (size 0.9 0.9)) (justify left)))
+(symbol (lib_id "TripTracer_V1:PWR_DIODE") (at 256.54 269.24 0) (unit 1) (in_bom yes) (on_board yes) (dnp no)
+(property "Reference" "D308" (at 256.54 252.73000000000002 0) (effects (font (size 1 1))))
+(property "Value" "BAS70-02V-HG3-08 EN FAILSAFE CLAMP" (at 256.54 255.27 0) (effects (font (size 1 1))))
+(property "Footprint" "Diode_SMD:D_SOD-523" (at 256.54 269.24 0) (effects (font (size 1 1)) (hide yes)))
+(property "MPN" "BAS70-02V-HG3-08" (at 0 0 0) (effects (font (size 1 1)) (hide yes)))
+(property "K_net" "VS_READY_RESET_OD_PRELIM" (at 0 0 0) (effects (font (size 1 1)) (hide yes)))
+(property "A_net" "CTRL_EN" (at 0 0 0) (effects (font (size 1 1)) (hide yes)))
+(pin "1")
+(pin "2")
+(instances (project "TripPower_5V2A" (path "/f1512578-cc72-4c26-bf70-dbbd00000001/f1512578-cc72-4c26-bf70-dbbd00000005" (reference "D308") (unit 1)))))
+(wire (pts (xy 246.38000000000002 269.24) (xy 241.3 269.24)) (stroke (width 0) (type default)))
+(global_label "VS_READY_RESET_OD_PRELIM" (shape bidirectional) (at 241.3 269.24 0) (effects (font (size 0.9 0.9)) (justify left)))
+(wire (pts (xy 266.70000000000005 269.24) (xy 271.78000000000003 269.24)) (stroke (width 0) (type default)))
+(global_label "CTRL_EN" (shape bidirectional) (at 271.78000000000003 269.24 0) (effects (font (size 0.9 0.9)) (justify left)))
 (embedded_fonts no))
