File: hardware/modules/TripPower_5V2A/02_5V_LMR38020.kicad_sch (KiCad schematic)
At the start: 12 parts, among them U101 LMR38020SQDDARQ1

Commit message: hardware(TripPower): align standalone sheet and symbol library to fuse-free protected-source auxiliary output
Connections:
- net VIN_PROTECTED_MAIN renamed VIN_PROTECTED_UNFUSED
Other:
- note added: "TripPower standalone: VIN_PROTECTED_UNFUSED is LM74930 common output, shared with an UNFUSED output pin; external branch cable fuse required; BUCK EN pin2 equals own VIN pin3. 5V_OUT pin is direct raw 2A output; no USB mux here. Do not fabricate: protection surge, thermals and FCH0650 provisional footprint unresolved."
- note removed: "TripPower standalone: VIN_PROTECTED_MAIN comes from separate LM74930 page; BUCK EN pin2 equals own VIN pin3. 5V_OUT pin is direct raw 2A output; no USB mux here. Do not fabricate: protection surge, thermals and FCH0650 provisional footprint unresolved."

Commit message: TripPower Weg A: use 15uH Bourns SRP7050TA AEC-Q200 in LMR38020 buck
Parts:
- L101: value 15uH FCH0650-150M Isat5.5A -> 15uH Bourns SRP7050TA-150M AEC-Q200; footprint Tripmaster:L_FANGCHENG_FCH0650_150M -> Tripmaster:L_BOURNS_SRP7050TA_150M; MPN FCH0650-150M -> SRP7050TA-150M
