File: hardware/modules/TripPower_5V2A/01_Protection_LM74930_D301_BACKUP_PROTOTYPE.kicad_sch (KiCad schematic)
At the start: 38 parts, among them J301 INPUT: VIN/RUN/GND, J302 OUT: PROT_UNFUSED/5V/GND, Q301 SQM10250E_GE3 250V CANDIDATE, Q302 BUK7Y4R8-60EX 60V CANDIDATE, U301 LM74930QRGERQ1

Commit message: Weg A prototype: specify stocked Comchip 5W AEC-Q101 SMC backup clamp D306 instead of 3W SMB
Parts:
- D306: value SZ1SMB5943BT3G 56V AEC-Q101 BACKUP PROTOTYPE -> ACZRC5370B-G 56V 5W AEC-Q101 BACKUP; footprint Diode_SMD:D_SMB -> Diode_SMD:D_SMC
Changed lines of the file:
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@@
 (symbol (lib_id "TripTracer_V1:PWR_CPOL") (at 149.86 325.12 0) (unit 1) (in_bom yes) (on_board yes) (dnp no) (property "Reference" "C306" (at 149.86 311.15 0) (effects (font (size 1 1)))) (property "Value" "47uF 63V POST SHUNT" (at 149.86 313.69 0) (effects (font (size 1 1)))) (property "Footprint" "Capacitor_SMD:CP_Elec_8x10.5" (at 149.86 325.12 0) (effects (font (size 1.0 1.0)) (hide yes))) (pin "1") (pin "2") (instances (project "TripPower_5V2A" (path "/f1512578-cc72-4c26-bf70-dbbd00000001/f1512578-cc72-4c26-bf70-dbbd00000002" (reference "C306") (unit 1)))))
 (symbol (lib_id "TripTracer_V1:PWR_DIODE") (at 234.95 325.12 0) (unit 1) (in_bom yes) (on_board yes) (dnp no) (property "Reference" "D301" (at 234.95 311.15 0) (effects (font (size 1 1)))) (property "Value" "1SMB5943BT3G 56V ZENER" (at 234.95 313.69 0) (effects (font (size 1 1)))) (property "Footprint" "Diode_SMD:D_SMB" (at 234.95 325.12 0) (effects (font (size 1.0 1.0)) (hide yes))) (pin "1") (pin "2") (instances (project "TripPower_5V2A" (path "/f1512578-cc72-4c26-bf70-dbbd00000001/f1512578-cc72-4c26-bf70-dbbd00000002" (reference "D301") (unit 1)))))
-(symbol (lib_id "TripTracer_V1:PWR_DIODE") (at 270.51 352.00 0) (unit 1) (in_bom yes) (on_board yes) (dnp no) (property "Reference" "D306" (at 270.51 338.03 0) (effects (font (size 1 1)))) (property "Value" "SZ1SMB5943BT3G 56V AEC-Q101 BACKUP PROTOTYPE" (at 270.51 340.57 0) (effects (font (size 1 1)))) (property "Footprint" "Diode_SMD:D_SMB" (at 270.51 352.00 0) (effects (font (size 1.0 1.0)) (hide yes))) (pin "1") (pin "2") (instances (project "TripPower_5V2A" (path "/f1512578-cc72-4c26-bf70-dbbd00000001/f1512578-cc72-4c26-bf70-dbbd00000002" (reference "D306") (unit 1)))))
+(symbol (lib_id "TripTracer_V1:PWR_DIODE") (at 270.51 352.00 0) (unit 1) (in_bom yes) (on_board yes) (dnp no) (property "Reference" "D306" (at 270.51 338.03 0) (effects (font (size 1 1)))) (property "Value" "ACZRC5370B-G 56V 5W AEC-Q101 BACKUP" (at 270.51 340.57 0) (effects (font (size 1 1)))) (property "Footprint" "Diode_SMD:D_SMC" (at 270.51 352.00 0) (effects (font (size 1.0 1.0)) (hide yes))) (pin "1") (pin "2") (instances (project "TripPower_5V2A" (path "/f1512578-cc72-4c26-bf70-dbbd00000001/f1512578-cc72-4c26-bf70-dbbd00000002" (reference "D306") (unit 1)))))
 (wire (pts (xy 255.27 352.00) (xy 260.35 352.00)) (stroke (width 0) (type default)))
 (global_label "VS_CLAMP" (shape bidirectional) (at 255.27 352.00 0) (effects (font (size 0.9 0.9)) (justify left)))

Commit message: Weg A: bind exact automotive D306 manufacturer MPN and datasheet in KiCad prototype
Parts:
- D306: MPN (none) -> ACZRC5370B-G
Changed lines of the file:
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@@
 (symbol (lib_id "TripTracer_V1:PWR_CPOL") (at 149.86 325.12 0) (unit 1) (in_bom yes) (on_board yes) (dnp no) (property "Reference" "C306" (at 149.86 311.15 0) (effects (font (size 1 1)))) (property "Value" "47uF 63V POST SHUNT" (at 149.86 313.69 0) (effects (font (size 1 1)))) (property "Footprint" "Capacitor_SMD:CP_Elec_8x10.5" (at 149.86 325.12 0) (effects (font (size 1.0 1.0)) (hide yes))) (pin "1") (pin "2") (instances (project "TripPower_5V2A" (path "/f1512578-cc72-4c26-bf70-dbbd00000001/f1512578-cc72-4c26-bf70-dbbd00000002" (reference "C306") (unit 1)))))
 (symbol (lib_id "TripTracer_V1:PWR_DIODE") (at 234.95 325.12 0) (unit 1) (in_bom yes) (on_board yes) (dnp no) (property "Reference" "D301" (at 234.95 311.15 0) (effects (font (size 1 1)))) (property "Value" "1SMB5943BT3G 56V ZENER" (at 234.95 313.69 0) (effects (font (size 1 1)))) (property "Footprint" "Diode_SMD:D_SMB" (at 234.95 325.12 0) (effects (font (size 1.0 1.0)) (hide yes))) (pin "1") (pin "2") (instances (project "TripPower_5V2A" (path "/f1512578-cc72-4c26-bf70-dbbd00000001/f1512578-cc72-4c26-bf70-dbbd00000002" (reference "D301") (unit 1)))))
-(symbol (lib_id "TripTracer_V1:PWR_DIODE") (at 270.51 352.00 0) (unit 1) (in_bom yes) (on_board yes) (dnp no) (property "Reference" "D306" (at 270.51 338.03 0) (effects (font (size 1 1)))) (property "Value" "ACZRC5370B-G 56V 5W AEC-Q101 BACKUP" (at 270.51 340.57 0) (effects (font (size 1 1)))) (property "Footprint" "Diode_SMD:D_SMC" (at 270.51 352.00 0) (effects (font (size 1.0 1.0)) (hide yes))) (pin "1") (pin "2") (instances (project "TripPower_5V2A" (path "/f1512578-cc72-4c26-bf70-dbbd00000001/f1512578-cc72-4c26-bf70-dbbd00000002" (reference "D306") (unit 1)))))
+(symbol (lib_id "TripTracer_V1:PWR_DIODE") (at 270.51 352.00 0) (unit 1) (in_bom yes) (on_board yes) (dnp no) (property "Reference" "D306" (at 270.51 338.03 0) (effects (font (size 1 1)))) (property "Value" "ACZRC5370B-G 56V 5W AEC-Q101 BACKUP" (at 270.51 340.57 0) (effects (font (size 1 1)))) (property "Footprint" "Diode_SMD:D_SMC" (at 270.51 352.00 0) (effects (font (size 1.0 1.0)) (hide yes))) (property "MPN" "ACZRC5370B-G" (at 0 0 0) (effects (font (size 1 1)) (hide yes))) (property "Datasheet" "https://www.comchiptech.com/admin/files/product/ACZRC53xxB-G%20Series%20RevD.pdf" (at 0 0 0) (effects (font (size 1 1)) (hide yes))) (pin "1") (pin "2") (instances (project "TripPower_5V2A" (path "/f1512578-cc72-4c26-bf70-dbbd00000001/f1512578-cc72-4c26-bf70-dbbd00000002" (reference "D306") (unit 1)))))
 (wire (pts (xy 255.27 352.00) (xy 260.35 352.00)) (stroke (width 0) (type default)))
 (global_label "VS_CLAMP" (shape bidirectional) (at 255.27 352.00 0) (effects (font (size 0.9 0.9)) (justify left)))
