File: hardware/modules/TripPower_5V2A/01_Protection_LM74930_Q301SHORT_CURRENTLIMIT_PROTOTYPE.kicad_sch (KiCad schematic)
At the start: 40 parts, among them J301 INPUT: VIN/RUN/GND, J302 OUT: PROT_UNFUSED/5V/GND, Q301 SQM10250E_GE3 250V CANDIDATE, Q302 BUK7Y4R8-60EX 60V CANDIDATE, Q307 BSP135H6327XTSA1 600V DEPL AE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, U301 LM74930QRGERQ1

Commit message: Weg A: choose AEC-Q200 Yageo AC1206FR-071K5L for 1.5k Q307 limit resistor
Parts:
- R342: MPN RC1206FR-071K5L -> AC1206FR-071K5L
Changed lines of the file:
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@@
 (global_label "GND" (shape bidirectional) (at 506.73 350.52 0) (effects (font (size 0.9 0.9)) (justify left)))
 (symbol (lib_id "TripTracer_V1:PWR_Q_HV") (at 100.33 383.54 0) (unit 1) (in_bom yes) (on_board yes) (dnp no) (property "Reference" "Q307" (at 100.33 369.57 0) (effects (font (size 1 1)))) (property "Value" "BSP135H6327XTSA1 600V DEPL AEC-Q101" (at 100.33 372.11 0) (effects (font (size 1 1)))) (property "Footprint" "Package_TO_SOT_SMD:SOT-223-3_TabPin2" (at 100.33 383.54 0) (effects (font (size 1.0 1.0)) (hide yes))) (property "MPN" "BSP135H6327XTSA1" (at 0 0 0) (effects (font (size 1 1)) (hide yes))) (property "Datasheet" "https://www.infineon.com/part/BSP135" (at 0 0 0) (effects (font (size 1 1)) (hide yes))) (pin "1") (pin "2") (pin "3") (instances (project "TripPower_5V2A" (path "/f1512578-cc72-4c26-bf70-dbbd00000001/f1512578-cc72-4c26-bf70-dbbd00000002" (reference "Q307") (unit 1)))))
-(symbol (lib_id "Tripmaster_Sym:R") (at 205.74 383.54 0) (unit 1) (in_bom yes) (on_board yes) (dnp no) (property "Reference" "R342" (at 205.74 369.57 0) (effects (font (size 1 1)))) (property "Value" "1.5k 1% 1206 SOURCE CURRENT LIMIT" (at 205.74 372.11 0) (effects (font (size 1 1)))) (property "Footprint" "Resistor_SMD:R_1206_3216Metric" (at 205.74 383.54 0) (effects (font (size 1.0 1.0)) (hide yes))) (property "MPN" "RC1206FR-071K5L" (at 0 0 0) (effects (font (size 1 1)) (hide yes))) (pin "1") (pin "2") (instances (project "TripPower_5V2A" (path "/f1512578-cc72-4c26-bf70-dbbd00000001/f1512578-cc72-4c26-bf70-dbbd00000002" (reference "R342") (unit 1)))))
+(symbol (lib_id "Tripmaster_Sym:R") (at 205.74 383.54 0) (unit 1) (in_bom yes) (on_board yes) (dnp no) (property "Reference" "R342" (at 205.74 369.57 0) (effects (font (size 1 1)))) (property "Value" "1.5k 1% 1206 SOURCE CURRENT LIMIT" (at 205.74 372.11 0) (effects (font (size 1 1)))) (property "Footprint" "Resistor_SMD:R_1206_3216Metric" (at 205.74 383.54 0) (effects (font (size 1.0 1.0)) (hide yes))) (property "MPN" "AC1206FR-071K5L" (at 0 0 0) (effects (font (size 1 1)) (hide yes))) (pin "1") (pin "2") (instances (project "TripPower_5V2A" (path "/f1512578-cc72-4c26-bf70-dbbd00000001/f1512578-cc72-4c26-bf70-dbbd00000002" (reference "R342") (unit 1)))))
 (wire (pts (xy 85.09 383.54) (xy 66.04 383.54)) (stroke (width 0) (type default)))
 (global_label "VS_CLAMP" (shape bidirectional) (at 66.04 383.54 0) (effects (font (size 0.9 0.9)) (justify left)))
