File: hardware/modules/TripPower_5V2A/01_Protection_LM74930_INDEPENDENT_AP74502_GUARD_PROTOTYPE.kicad_sch (KiCad schematic)
At the start: 49 parts, among them J301 INPUT: VIN/RUN/GND, J302 OUT: PROT_UNFUSED/5V/GND, Q301 SQM10250E_GE3 250V CANDIDATE, Q302 BUK7Y4R8-60EX 60V CANDIDATE, Q401 SQM10250E_GE3 250V INDEPENDEN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, U301 LM74930QRGERQ1, U401 AP74502HQTA8-7

Commit message: Weg A independent guard: correct AP74502 EN1/VIN and GND2 polarised pin labels before native ERC
Connections:
- net AP_VIN_CLAMP: now also U401.1 (EN/UVLO); no longer U401.2 (GND)
- net GND: now also U401.2 (GND); no longer U401.1 (EN/UVLO)
Changed lines of the file:
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@@
 (instances (project "TripPower_5V2A" (path "/f1512578-cc72-4c26-bf70-dbbd00000001/f1512578-cc72-4c26-bf70-dbbd00000002" (reference "U401") (unit 1)))))
 (wire (pts (xy 528.32 370.84) (xy 523.24 370.84)) (stroke (width 0) (type default)))
-(global_label "GND" (shape bidirectional) (at 523.24 370.84 0) (effects (font (size 0.9 0.9)) (justify left)))
+(global_label "AP_VIN_CLAMP" (shape bidirectional) (at 523.24 370.84 0) (effects (font (size 0.9 0.9)) (justify left)))
 (wire (pts (xy 528.32 396.24) (xy 523.24 396.24)) (stroke (width 0) (type default)))
-(global_label "AP_VIN_CLAMP" (shape bidirectional) (at 523.24 396.24 0) (effects (font (size 0.9 0.9)) (justify left)))
+(global_label "GND" (shape bidirectional) (at 523.24 396.24 0) (effects (font (size 0.9 0.9)) (justify left)))
 (wire (pts (xy 574.04 370.84) (xy 579.12 370.84)) (stroke (width 0) (type default)))
 (global_label "AP_VCAP" (shape bidirectional) (at 579.12 370.84 0) (effects (font (size 0.9 0.9)) (justify left)))

Commit message: Weg A AP guard: choose stocked automotive 10k OV bottom for robust 30V recovery margin
Parts:
- R407: value 10.5k 1% OV BOTTOM -> 10k 1% OV BOTTOM; MPN AC1206FR-0710K5L -> AC1206FR-0710KL
Changed lines of the file:
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@@
 (symbol (lib_id "Tripmaster_Sym:R") (at 400.05 383.54 0) (unit 1) (in_bom yes) (on_board yes) (dnp no) (property "Reference" "R405" (at 400.05 369.57 0) (effects (font (size 1 1)))) (property "Value" "100k 1% OV TOP 2" (at 400.05 372.11 0) (effects (font (size 1 1)))) (property "Footprint" "Resistor_SMD:R_1206_3216Metric" (at 400.05 383.54 0) (effects (font (size 1.0 1.0)) (hide yes))) (property "MPN" "AC1206FR-07100KL" (at 0 0 0) (effects (font (size 1 1)) (hide yes))) (pin "1") (pin "2") (instances (project "TripPower_5V2A" (path "/f1512578-cc72-4c26-bf70-dbbd00000001/f1512578-cc72-4c26-bf70-dbbd00000002" (reference "R405") (unit 1)))))
 (symbol (lib_id "Tripmaster_Sym:R") (at 440.69 383.54 0) (unit 1) (in_bom yes) (on_board yes) (dnp no) (property "Reference" "R406" (at 440.69 369.57 0) (effects (font (size 1 1)))) (property "Value" "100k 1% OV TOP 3" (at 440.69 372.11 0) (effects (font (size 1 1)))) (property "Footprint" "Resistor_SMD:R_1206_3216Metric" (at 440.69 383.54 0) (effects (font (size 1.0 1.0)) (hide yes))) (property "MPN" "AC1206FR-07100KL" (at 0 0 0) (effects (font (size 1 1)) (hide yes))) (pin "1") (pin "2") (instances (project "TripPower_5V2A" (path "/f1512578-cc72-4c26-bf70-dbbd00000001/f1512578-cc72-4c26-bf70-dbbd00000002" (reference "R406") (unit 1)))))
-(symbol (lib_id "Tripmaster_Sym:R") (at 481.33 383.54 0) (unit 1) (in_bom yes) (on_board yes) (dnp no) (property "Reference" "R407" (at 481.33 369.57 0) (effects (font (size 1 1)))) (property "Value" "10.5k 1% OV BOTTOM" (at 481.33 372.11 0) (effects (font (size 1 1)))) (property "Footprint" "Resistor_SMD:R_1206_3216Metric" (at 481.33 383.54 0) (effects (font (size 1.0 1.0)) (hide yes))) (property "MPN" "AC1206FR-0710K5L" (at 0 0 0) (effects (font (size 1 1)) (hide yes))) (pin "1") (pin "2") (instances (project "TripPower_5V2A" (path "/f1512578-cc72-4c26-bf70-dbbd00000001/f1512578-cc72-4c26-bf70-dbbd00000002" (reference "R407") (unit 1)))))
+(symbol (lib_id "Tripmaster_Sym:R") (at 481.33 383.54 0) (unit 1) (in_bom yes) (on_board yes) (dnp no) (property "Reference" "R407" (at 481.33 369.57 0) (effects (font (size 1 1)))) (property "Value" "10k 1% OV BOTTOM" (at 481.33 372.11 0) (effects (font (size 1 1)))) (property "Footprint" "Resistor_SMD:R_1206_3216Metric" (at 481.33 383.54 0) (effects (font (size 1.0 1.0)) (hide yes))) (property "MPN" "AC1206FR-0710KL" (at 0 0 0) (effects (font (size 1 1)) (hide yes))) (pin "1") (pin "2") (instances (project "TripPower_5V2A" (path "/f1512578-cc72-4c26-bf70-dbbd00000001/f1512578-cc72-4c26-bf70-dbbd00000002" (reference "R407") (unit 1)))))
 (symbol (lib_id "TripTracer_V1:PWR_DIODE") (at 237.49 383.54 0) (unit 1) (in_bom yes) (on_board yes) (dnp no) (property "Reference" "D401" (at 237.49 369.57 0) (effects (font (size 1 1)))) (property "Value" "1SMB5943BT3G 56V AP VIN ZENER" (at 237.49 372.11 0) (effects (font (size 1 1)))) (property "Footprint" "Diode_SMD:D_SMB" (at 237.49 383.54 0) (effects (font (size 1.0 1.0)) (hide yes))) (property "MPN" "1SMB5943BT3G" (at 0 0 0) (effects (font (size 1 1)) (hide yes))) (pin "1") (pin "2") (instances (project "TripPower_5V2A" (path "/f1512578-cc72-4c26-bf70-dbbd00000001/f1512578-cc72-4c26-bf70-dbbd00000002" (reference "D401") (unit 1)))))
 (symbol (lib_id "Tripmaster_Sym:C") (at 278.13 383.54 0) (unit 1) (in_bom yes) (on_board yes) (dnp no) (property "Reference" "C401" (at 278.13 369.57 0) (effects (font (size 1 1)))) (property "Value" "1uF 100V AP VIN RESERVOIR" (at 278.13 372.11 0) (effects (font (size 1 1)))) (property "Footprint" "Capacitor_SMD:C_1210_3225Metric" (at 278.13 383.54 0) (effects (font (size 1.0 1.0)) (hide yes))) (property "MPN" "C1210C105K1RACAUTO" (at 0 0 0) (effects (font (size 1 1)) (hide yes))) (property "Supplier_URL" "https://www.mouser.de/ProductDetail/KEMET/C1210C105K1RACAUTO" (at 0 0 0) (effects (font (size 1 1)) (hide yes))) (pin "1") (pin "2") (instances (project "TripPower_5V2A" (path "/f1512578-cc72-4c26-bf70-dbbd00000001/f1512578-cc72-4c26-bf70-dbbd00000002" (reference "C401") (unit 1)))))

Commit message: Weg A AP guard: portable KiCad10 AP symbol + explicit nonpopulated R-fed VIN PWR flag fixes native ERC without lying about populated hardware
Parts:
- U401: symbol TripPower_A:AP74502HQ_SOT28 -> TripPower_AP74502:AP74502HQ_SOT28
Changed lines of the file:
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@@
 (wire (pts (xy 492.76 383.54) (xy 497.84 383.54)) (stroke (width 0) (type default)))
 (global_label "GND" (shape bidirectional) (at 497.84 383.54 0) (effects (font (size 0.9 0.9)) (justify left)))
-(symbol (lib_id "TripPower_A:AP74502HQ_SOT28") (at 551.18 383.54 0) (unit 1) (in_bom yes) (on_board yes) (dnp no)
+(symbol (lib_id "TripPower_AP74502:AP74502HQ_SOT28") (at 551.18 383.54 0) (unit 1) (in_bom yes) (on_board yes) (dnp no)
 (property "Reference" "U401" (at 551.18 362.00 0) (effects (font (size 1 1))))
 (property "Value" "AP74502HQTA8-7" (at 551.18 364.54 0) (effects (font (size 1 1))))
@@
 (wire (pts (xy 574.04 396.24) (xy 579.12 396.24)) (stroke (width 0) (type default)))
 (global_label "VIN_A_GUARD_OUT" (shape bidirectional) (at 579.12 396.24 0) (effects (font (size 0.9 0.9)) (justify left)))
+(symbol (lib_id "TripPower_AP74502:AP_VIN_FEED_FLAG") (at 551.18 350.52 0) (unit 1) (in_bom no) (on_board no) (dnp no)
+(property "Reference" "#FLG401" (at 551.18 345.44 0) (effects (font (size 1 1)) (hide yes)))
+(property "Value" "AP_VIN_FEED_FLAG" (at 551.18 354.33 0) (effects (font (size 1 1)) (hide yes)))
+(pin "1")
+(instances (project "TripPower_5V2A" (path "/f1512578-cc72-4c26-bf70-dbbd00000001/f1512578-cc72-4c26-bf70-dbbd00000002" (reference "#FLG401") (unit 1)))))
+(wire (pts (xy 551.18 350.52) (xy 556.26 350.52)) (stroke (width 0) (type default)))
+(global_label "AP_VIN_CLAMP" (shape bidirectional) (at 556.26 350.52 0) (effects (font (size 0.9 0.9)) (justify left)))
 (embedded_fonts no))
