File: hardware/modules/TripPower_5V2A/02_5V_LMR38020_PGOOD_BACKUP_INTERFACE_PROTOTYPE.kicad_sch (KiCad schematic)
At the start: 15 parts, among them Q501 BVSS123LT1G PGOOD STATUS OPEN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, U101 LMR38020SQDDARQ1

Commit message: Weg A R6: connect PWR_FAIL collector to non-BOM physical TP501 signal pad and eliminate orphan ERC label
Parts:
- added TP501: PWR_FAIL_SIGNAL_PAD, TestPoint:TestPoint_Pad_1.5x1.5mm, symbol TripPower_PGOOD:SignalPad
Connections:
- net PWR_OK_SINK_FAIL_RELEASE: now also TP501.1 (PAD)
