File: hardware/modules/TripPower_REV6_A/01_TPS26631_REV6.kicad_sch (KiCad schematic)
At the start: 13 parts, among them Q201 SQM100N10-10_GE3 100V AEC, Q202 BSS138LT1G DRIVER PULLDOWN, U201 TPS26631PWPR

Commit message: Weg A REV6: widen certified 10V-start UVLO margin with 810k/100k/33.2k OV divider; keep OV >32 <36
Parts:
- R201: value 820k 1pct UV_TOP -> 810k 1pct UV_TOP; MPN AC1206FR-07820KL -> AC1206FR-07810KL
- R202: value 86.6k 1pct UV_MID -> 100k 1pct UV_MID; MPN AC1206FR-0786K6L -> AC1206FR-07100KL
Other:
- note added: "R201=810k R202=100k R203=33k2: OVP rising around 34.1V typical, UVLO rising around 8.5V typical. Need verify OVP leak/TCR/tol, 10V loaded start, 32V survival; not production. No extra 200V high voltage network."
- note removed: "R201=820k R202=86k6 R203=33k2: OVP top 33.97V typical, UVLO rising 9.42V typical. Need verify OVP leak/TCR/tol, 10V loaded start, 32V survival; not production. No extra 200V high voltage network."
Changed lines of the file:
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@@
 (title_block (title "TripPower REV6 A - TPS26631 60V eFuse and 100V reverse FET") (date "2026-10-15") (rev "SCHEMATIC EXPERIMENT / NO FAB"))
 (text "TI TPS26631 PWPR Fig9-2-derived power stage: 10..32V; OV <=36 via R201..203, 58V 350ms only certified conditioned input <60V incl ringing. ILIM nominal3A. Q201 body diode orientation, Q202 fast off, external F_MAIN. TPS26631 industrial NOT AEC, thermals/ESD/RAW/USB/open-pin/temperature NOT qualified." (at 27.94 34.29 0) (effects (font (size 1.016 1.016))))
-(text "R201=820k R202=86k6 R203=33k2: OVP top 33.97V typical, UVLO rising 9.42V typical. Need verify OVP leak/TCR/tol, 10V loaded start, 32V survival; not production. No extra 200V high voltage network." (at 27.94 43.18 0) (effects (font (size 1.016 1.016))))
+(text "R201=810k R202=100k R203=33k2: OVP rising around 34.1V typical, UVLO rising around 8.5V typical. Need verify OVP leak/TCR/tol, 10V loaded start, 32V survival; not production. No extra 200V high voltage network." (at 27.94 43.18 0) (effects (font (size 1.016 1.016))))
 (text "WARNING: 58V at connector must already include wiring overshoots. eFuse ABS 67V, MAX recommended 60V. TMP 85C safe-off not implemented, must be implemented before FAB. RAW testpad not 0.5A-rated connector." (at 27.94 50.8 0) (effects (font (size 1.016 1.016))))
 (symbol (lib_id "TripPower_REV6:TPS26631_PWP20") (at 248.92 127 0) (unit 1) (in_bom yes) (on_board yes) (dnp no)
@@
 (symbol (lib_id "Tripmaster_Sym:R") (at 64.77 205.74 0) (unit 1) (in_bom yes) (on_board yes) (dnp no)
 (property "Reference" "R201" (at 64.77 189.74 0) (effects (font (size 1 1))))
-(property "Value" "820k 1pct UV_TOP" (at 64.77 192.74 0) (effects (font (size 1 1))))
+(property "Value" "810k 1pct UV_TOP" (at 64.77 192.74 0) (effects (font (size 1 1))))
 (property "Footprint" "Resistor_SMD:R_1206_3216Metric" (at 64.77 205.74 0) (effects (font (size 1 1)) (hide yes)))
-(property "MPN" "AC1206FR-07820KL" (at 0 0 0) (effects (font (size 1 1)) (hide yes)))
+(property "MPN" "AC1206FR-07810KL" (at 0 0 0) (effects (font (size 1 1)) (hide yes)))
 (pin "1")
 (pin "2")
@@
 (symbol (lib_id "Tripmaster_Sym:R") (at 116.84 205.74 0) (unit 1) (in_bom yes) (on_board yes) (dnp no)
 (property "Reference" "R202" (at 116.84 189.74 0) (effects (font (size 1 1))))
-(property "Value" "86.6k 1pct UV_MID" (at 116.84 192.74 0) (effects (font (size 1 1))))
+(property "Value" "100k 1pct UV_MID" (at 116.84 192.74 0) (effects (font (size 1 1))))
 (property "Footprint" "Resistor_SMD:R_1206_3216Metric" (at 116.84 205.74 0) (effects (font (size 1 1)) (hide yes)))
-(property "MPN" "AC1206FR-0786K6L" (at 0 0 0) (effects (font (size 1 1)) (hide yes)))
+(property "MPN" "AC1206FR-07100KL" (at 0 0 0) (effects (font (size 1 1)) (hide yes)))
 (pin "1")
 (pin "2")

Commit message: Weg A REV6: 402k/49.9k/16.5k UV/OV chain; model worst OVP 32.34-35.86 incl leakage & hot TCR
Parts:
- R201: value 810k 1pct UV_TOP -> 402k 1pct UV_TOP; MPN AC1206FR-07810KL -> AC1206FR-07402KL
- R202: value 100k 1pct UV_MID -> 49.9k 1pct UV_MID; MPN AC1206FR-07100KL -> AC1206FR-0749K9L
- R203: value 33.2k 1pct OV_BOT -> 16.5k 1pct OV_BOT; MPN AC1206FR-0733K2L -> AC1206FR-0716K5L
Other:
- note added: "R201=402k R202=49k9 R203=16k5: OV rise 34.07V typ / 32.34..35.86V modeled limits, UV rise 8.47V typ. Need verify OVP leak/TCR/tol, 10V loaded start, 32V survival; not production. No extra 200V high voltage network."
- note removed: "R201=810k R202=100k R203=33k2: OVP rising around 34.1V typical, UVLO rising around 8.5V typical. Need verify OVP leak/TCR/tol, 10V loaded start, 32V survival; not production. No extra 200V high voltage network."
Changed lines of the file:
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@@
 (title_block (title "TripPower REV6 A - TPS26631 60V eFuse and 100V reverse FET") (date "2026-10-15") (rev "SCHEMATIC EXPERIMENT / NO FAB"))
 (text "TI TPS26631 PWPR Fig9-2-derived power stage: 10..32V; OV <=36 via R201..203, 58V 350ms only certified conditioned input <60V incl ringing. ILIM nominal3A. Q201 body diode orientation, Q202 fast off, external F_MAIN. TPS26631 industrial NOT AEC, thermals/ESD/RAW/USB/open-pin/temperature NOT qualified." (at 27.94 34.29 0) (effects (font (size 1.016 1.016))))
-(text "R201=810k R202=100k R203=33k2: OVP rising around 34.1V typical, UVLO rising around 8.5V typical. Need verify OVP leak/TCR/tol, 10V loaded start, 32V survival; not production. No extra 200V high voltage network." (at 27.94 43.18 0) (effects (font (size 1.016 1.016))))
+(text "R201=402k R202=49k9 R203=16k5: OV rise 34.07V typ / 32.34..35.86V modeled limits, UV rise 8.47V typ. Need verify OVP leak/TCR/tol, 10V loaded start, 32V survival; not production. No extra 200V high voltage network." (at 27.94 43.18 0) (effects (font (size 1.016 1.016))))
 (text "WARNING: 58V at connector must already include wiring overshoots. eFuse ABS 67V, MAX recommended 60V. TMP 85C safe-off not implemented, must be implemented before FAB. RAW testpad not 0.5A-rated connector." (at 27.94 50.8 0) (effects (font (size 1.016 1.016))))
 (symbol (lib_id "TripPower_REV6:TPS26631_PWP20") (at 248.92 127 0) (unit 1) (in_bom yes) (on_board yes) (dnp no)
@@
 (symbol (lib_id "Tripmaster_Sym:R") (at 64.77 205.74 0) (unit 1) (in_bom yes) (on_board yes) (dnp no)
 (property "Reference" "R201" (at 64.77 189.74 0) (effects (font (size 1 1))))
-(property "Value" "810k 1pct UV_TOP" (at 64.77 192.74 0) (effects (font (size 1 1))))
+(property "Value" "402k 1pct UV_TOP" (at 64.77 192.74 0) (effects (font (size 1 1))))
 (property "Footprint" "Resistor_SMD:R_1206_3216Metric" (at 64.77 205.74 0) (effects (font (size 1 1)) (hide yes)))
-(property "MPN" "AC1206FR-07810KL" (at 0 0 0) (effects (font (size 1 1)) (hide yes)))
+(property "MPN" "AC1206FR-07402KL" (at 0 0 0) (effects (font (size 1 1)) (hide yes)))
 (pin "1")
 (pin "2")
@@
 (symbol (lib_id "Tripmaster_Sym:R") (at 116.84 205.74 0) (unit 1) (in_bom yes) (on_board yes) (dnp no)
 (property "Reference" "R202" (at 116.84 189.74 0) (effects (font (size 1 1))))
-(property "Value" "100k 1pct UV_MID" (at 116.84 192.74 0) (effects (font (size 1 1))))
+(property "Value" "49.9k 1pct UV_MID" (at 116.84 192.74 0) (effects (font (size 1 1))))
 (property "Footprint" "Resistor_SMD:R_1206_3216Metric" (at 116.84 205.74 0) (effects (font (size 1 1)) (hide yes)))
-(property "MPN" "AC1206FR-07100KL" (at 0 0 0) (effects (font (size 1 1)) (hide yes)))
+(property "MPN" "AC1206FR-0749K9L" (at 0 0 0) (effects (font (size 1 1)) (hide yes)))
 (pin "1")
 (pin "2")
@@
 (symbol (lib_id "Tripmaster_Sym:R") (at 167.64 205.74 0) (unit 1) (in_bom yes) (on_board yes) (dnp no)
 (property "Reference" "R203" (at 167.64 189.74 0) (effects (font (size 1 1))))
-(property "Value" "33.2k 1pct OV_BOT" (at 167.64 192.74 0) (effects (font (size 1 1))))
+(property "Value" "16.5k 1pct OV_BOT" (at 167.64 192.74 0) (effects (font (size 1 1))))
 (property "Footprint" "Resistor_SMD:R_1206_3216Metric" (at 167.64 205.74 0) (effects (font (size 1 1)) (hide yes)))
-(property "MPN" "AC1206FR-0733K2L" (at 0 0 0) (effects (font (size 1 1)) (hide yes)))
+(property "MPN" "AC1206FR-0716K5L" (at 0 0 0) (effects (font (size 1 1)) (hide yes)))
 (pin "1")
 (pin "2")
