File: hardware/modules/TripPower_REV6_A/01_TPS26631_REV6_FACTORY_OVP.kicad_sch (KiCad schematic)
At the start: 11 parts, among them Q201 SQM100N10-10_GE3 100V AEC, Q202 BSS138LT1G DRIVER PULLDOWN, U201 TPS26631PWPR

Commit message: TripPower A REV6 Round5: retain A23 auto-retry, document PGTH 1x limit and host safety gaps; fix KiCad OV notes, add independent CI gates; NO FAB
Other:
- note added: "R201=330k UVLO/no external rising divider, Yageo AC1206FR-07330KL 1pct/100ppm: at -20..+70C Rmin325.215k (> TI300k). TI factory OVP rising 33.2..35.4V/falling32.7..35.0V; 32V recovery margin min0.7V AT IN_SYS only, no ringing budget. 10V 5V2A+RAW startup and 58V pad stress NOT proven; A24 divider optional research only."
- note added: "TI TPS26631PWPR A23: 10..32V; factory OVP8=GND rising33.2..35.4V/falling32.7..35.0V; R201330k IN_SYS6->UVLO7. 58V/350ms at M8 does NOT guarantee <=60V at U201 pads. MODE12=GND auto retry; PGTH16=GND disables fast restart AND PGOOD HIGH/2x IOL burst; softstart via C203. SHDN13 OPEN (internal ON, ABS5.5V). RAW selective OCP/+85C safety/USB/ACC NOT implemented here. NO FAB."
- note removed: "R201=330k UVLO/no external rising divider; factory OVP8=GND Yageo RT 0.1pct/25ppm: OVP rising 32.223..33.880V, falling 29.864..31.833V, UV rising max8.822V; 32V static hysteresis margin0.167V. Need verify OVP leak/TCR/tol, 10V loaded start, 32V survival; not production. No extra 200V high voltage network."
- note removed: "TI TPS26631 PWPR Fig9-2-derived power stage: 10..32V; OV <=36 via R201..203, 58V 350ms only certified conditioned input <60V incl ringing. ILIM nominal3A. SHDN13 floats per TI internal pull-up, MUST NOT connect to 58V (ABS max5.5V). Q201 body diode orientation, Q202 fast off, external F_MAIN. TPS26631 industrial NOT AEC, thermals/ESD/RAW/USB/open-pin/temperature NOT qualified."
- title: TripPower REV6 A - TPS26631 60V eFuse and 100V reverse FET -> TripPower REV6 A23 - TPS26631 factory OVP, 330k UVLO
Changed lines of the file:
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@@
 (kicad_sch (version 20250114) (generator "eeschema") (paper "A3")
-(title_block (title "TripPower REV6 A - TPS26631 60V eFuse and 100V reverse FET") (date "2026-10-15") (rev "SCHEMATIC EXPERIMENT / NO FAB"))
-(text "TI TPS26631 PWPR Fig9-2-derived power stage: 10..32V; OV <=36 via R201..203, 58V 350ms only certified conditioned input <60V incl ringing. ILIM nominal3A. SHDN13 floats per TI internal pull-up, MUST NOT connect to 58V (ABS max5.5V). Q201 body diode orientation, Q202 fast off, external F_MAIN. TPS26631 industrial NOT AEC, thermals/ESD/RAW/USB/open-pin/temperature NOT qualified." (at 27.94 34.29 0) (effects (font (size 1.016 1.016))))
-(text "R201=330k UVLO/no external rising divider; factory OVP8=GND Yageo RT 0.1pct/25ppm: OVP rising 32.223..33.880V, falling 29.864..31.833V, UV rising max8.822V; 32V static hysteresis margin0.167V. Need verify OVP leak/TCR/tol, 10V loaded start, 32V survival; not production. No extra 200V high voltage network." (at 27.94 43.18 0) (effects (font (size 1.016 1.016))))
+(title_block (title "TripPower REV6 A23 - TPS26631 factory OVP, 330k UVLO") (date "2026-10-15") (rev "SCHEMATIC EXPERIMENT / NO FAB"))
+(text "TI TPS26631PWPR A23: 10..32V; factory OVP8=GND rising33.2..35.4V/falling32.7..35.0V; R201330k IN_SYS6->UVLO7. 58V/350ms at M8 does NOT guarantee <=60V at U201 pads. MODE12=GND auto retry; PGTH16=GND disables fast restart AND PGOOD HIGH/2x IOL burst; softstart via C203. SHDN13 OPEN (internal ON, ABS5.5V). RAW selective OCP/+85C safety/USB/ACC NOT implemented here. NO FAB." (at 27.94 34.29 0) (effects (font (size 1.016 1.016))))
+(text "R201=330k UVLO/no external rising divider, Yageo AC1206FR-07330KL 1pct/100ppm: at -20..+70C Rmin325.215k (> TI300k). TI factory OVP rising 33.2..35.4V/falling32.7..35.0V; 32V recovery margin min0.7V AT IN_SYS only, no ringing budget. 10V 5V2A+RAW startup and 58V pad stress NOT proven; A24 divider optional research only." (at 27.94 43.18 0) (effects (font (size 1.016 1.016))))
 (text "WARNING: 58V at connector must already include wiring overshoots. eFuse ABS 67V, MAX recommended 60V. TMP 85C safe-off not implemented, must be implemented before FAB. RAW testpad not 0.5A-rated connector." (at 27.94 50.8 0) (effects (font (size 1.016 1.016))))
 (symbol (lib_id "TripPower_REV6:TPS26631_PWP20") (at 248.92 127 0) (unit 1) (in_bom yes) (on_board yes) (dnp no)
