File: hardware/kicad/TripTracer_A23_Integration/04_ESP32_USB.kicad_sch (KiCad schematic)
At the start: 13 parts, among them J201 GCT USB4105-GF-A, U201 ESP32-S3-MINI-1-N8

Commit message: TripPower A23 integrated LAB: actually wire host PWR_FAIL 10k AEC-Q200 3V3 pullup to ESP32 GPIO1 and Q501 open drain
Connections:
- net PWR_OK_SINK_FAIL_RELEASE: now reaches U201.5 (IO1)
- no-connect marks 35 -> 34
Changed lines of the file:
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@@
 (wire (pts (xy 300.99 182.88) (xy 311.15 182.88)) (stroke (width 0) (type default)))
 (text "33 unused GPIOs deliberately marked NC in this LAB-only host sheet; FRAM/SD/GNSS/display circuits remain unimplemented. Not production-ready." (at 209.55 25.4 0) (effects (font (size 1.27 1.27))))
-(no_connect (at 311.15 60.96))
 (no_connect (at 311.15 66.04))
 (no_connect (at 311.15 71.12))
@@
 (no_connect (at 311.15 243.84))
 (no_connect (at 311.15 248.92))
+(global_label "PWR_OK_SINK_FAIL_RELEASE" (shape input) (at 311.15 60.96 0) (effects (font (size 1.016 1.016)) (justify left)))
 )
