File: hardware/kicad/TripTracer_A23_Integration/01_TPS26631_A23_INTEGRATED.kicad_sch (KiCad schematic)
At the start: 11 parts, among them Q941 SQM100N10-10_GE3 100V AEC, Q942 BSS138LT1G DRIVER PULLDOWN, U921 TPS26631PWPR

Commit message: TripPower A23 integrated lab: add physical no-BOM scope pads EFUSE_IN BGATE DRV OUT/buck VIN UVLO dVdT for 58V qualification
Parts:
- added TP944: EFUSE_IN before Q941 reverse MOSFET, TestPoint:TestPoint_Pad_1.5x1.5mm, symbol TripPower_PGOOD:SignalPad
- added TP945: Q941 BGATE to IN_SYS differential, TestPoint:TestPoint_Pad_1.5x1.5mm, symbol TripPower_PGOOD:SignalPad
- added TP946: Q942 DRV relative to IN_SYS, TestPoint:TestPoint_Pad_1.5x1.5mm, symbol TripPower_PGOOD:SignalPad
- added TP947: TPS OUT + buck VIN / shared RAW input, TestPoint:TestPoint_Pad_1.5x1.5mm, symbol TripPower_PGOOD:SignalPad
- added TP948: U921 UVLO sense to IN_SYS via R941, TestPoint:TestPoint_Pad_1.5x1.5mm, symbol TripPower_PGOOD:SignalPad
- added TP949: U921 dVdT - LOW voltage sense, TestPoint:TestPoint_Pad_1.5x1.5mm, symbol TripPower_PGOOD:SignalPad
Connections:
- net EFUSE_IN: now also TP944.1 (PAD)
- net R6_B_GATE: now also TP945.1 (PAD)
- net R6_DRV: now also TP946.1 (PAD)
- net R6_DVDT: now also TP949.1 (PAD)
- net UVLO_SENSE: now also TP948.1 (PAD)
- net VIN_PROTECTED_UNFUSED: now also TP947.1 (PAD)
Other:
- note added: "ROUND6 LAB ONLY: these pads are not in the original 23-position A23 project; inspect probe capacitance and differential pin limits at 58V. No unqualified PCB production."
Changed lines of the file:
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@@
 (wire (pts (xy 344.17 248.92) (xy 349.25 248.92)) (stroke (width 0) (type default)))
 (global_label "GND" (shape bidirectional) (at 349.25 248.92 0) (effects (font (size 1 1)) (justify left)))
-(embedded_fonts no))
+(symbol (lib_id "TripPower_PGOOD:SignalPad") (at 355.6 152.4 0) (unit 1) (in_bom no) (on_board yes) (dnp no)
+(property "Reference" "TP944" (at 355.6 136.4 0) (effects (font (size 1 1))))
+(property "Value" "EFUSE_IN before Q941 reverse MOSFET" (at 355.6 139.4 0) (effects (font (size 1 1))))
+(property "Footprint" "TestPoint:TestPoint_Pad_1.5x1.5mm" (at 355.6 152.4 0) (effects (font (size 1 1)) (hide yes)))
+(pin "1")
+(instances (project "TripTracer_A23_Integration" (path "/a26d9b0c-7f10-4e5a-a65f-000000000064/a26d9b0c-7f10-4e5a-a65f-000000000065" (reference "TP944") (unit 1)))))
+(global_label "EFUSE_IN" (shape bidirectional) (at 350.52 152.4 0) (effects (font (size 1 1)) (justify left)))
+(symbol (lib_id "TripPower_PGOOD:SignalPad") (at 355.6 165.1 0) (unit 1) (in_bom no) (on_board yes) (dnp no)
+(property "Reference" "TP945" (at 355.6 149.1 0) (effects (font (size 1 1))))
+(property "Value" "Q941 BGATE to IN_SYS differential" (at 355.6 152.1 0) (effects (font (size 1 1))))
+(property "Footprint" "TestPoint:TestPoint_Pad_1.5x1.5mm" (at 355.6 165.1 0) (effects (font (size 1 1)) (hide yes)))
+(pin "1")
+(instances (project "TripTracer_A23_Integration" (path "/a26d9b0c-7f10-4e5a-a65f-000000000064/a26d9b0c-7f10-4e5a-a65f-000000000065" (reference "TP945") (unit 1)))))
+(global_label "R6_B_GATE" (shape bidirectional) (at 350.52 165.1 0) (effects (font (size 1 1)) (justify left)))
+(symbol (lib_id "TripPower_PGOOD:SignalPad") (at 355.6 177.8 0) (unit 1) (in_bom no) (on_board yes) (dnp no)
+(property "Reference" "TP946" (at 355.6 161.8 0) (effects (font (size 1 1))))
+(property "Value" "Q942 DRV relative to IN_SYS" (at 355.6 164.8 0) (effects (font (size 1 1))))
+(property "Footprint" "TestPoint:TestPoint_Pad_1.5x1.5mm" (at 355.6 177.8 0) (effects (font (size 1 1)) (hide yes)))
+(pin "1")
+(instances (project "TripTracer_A23_Integration" (path "/a26d9b0c-7f10-4e5a-a65f-000000000064/a26d9b0c-7f10-4e5a-a65f-000000000065" (reference "TP946") (unit 1)))))
+(global_label "R6_DRV" (shape bidirectional) (at 350.52 177.8 0) (effects (font (size 1 1)) (justify left)))
+(symbol (lib_id "TripPower_PGOOD:SignalPad") (at 355.6 190.5 0) (unit 1) (in_bom no) (on_board yes) (dnp no)
+(property "Reference" "TP947" (at 355.6 174.5 0) (effects (font (size 1 1))))
+(property "Value" "TPS OUT + buck VIN / shared RAW input" (at 355.6 177.5 0) (effects (font (size 1 1))))
+(property "Footprint" "TestPoint:TestPoint_Pad_1.5x1.5mm" (at 355.6 190.5 0) (effects (font (size 1 1)) (hide yes)))
+(pin "1")
+(instances (project "TripTracer_A23_Integration" (path "/a26d9b0c-7f10-4e5a-a65f-000000000064/a26d9b0c-7f10-4e5a-a65f-000000000065" (reference "TP947") (unit 1)))))
+(global_label "VIN_PROTECTED_UNFUSED" (shape bidirectional) (at 350.52 190.5 0) (effects (font (size 1 1)) (justify left)))
+(symbol (lib_id "TripPower_PGOOD:SignalPad") (at 355.6 203.2 0) (unit 1) (in_bom no) (on_board yes) (dnp no)
+(property "Reference" "TP948" (at 355.6 187.2 0) (effects (font (size 1 1))))
+(property "Value" "U921 UVLO sense to IN_SYS via R941" (at 355.6 190.2 0) (effects (font (size 1 1))))
+(property "Footprint" "TestPoint:TestPoint_Pad_1.5x1.5mm" (at 355.6 203.2 0) (effects (font (size 1 1)) (hide yes)))
+(pin "1")
+(instances (project "TripTracer_A23_Integration" (path "/a26d9b0c-7f10-4e5a-a65f-000000000064/a26d9b0c-7f10-4e5a-a65f-000000000065" (reference "TP948") (unit 1)))))
+(global_label "UVLO_SENSE" (shape bidirectional) (at 350.52 203.2 0) (effects (font (size 1 1)) (justify left)))
+(symbol (lib_id "TripPower_PGOOD:SignalPad") (at 355.6 215.9 0) (unit 1) (in_bom no) (on_board yes) (dnp no)
+(property "Reference" "TP949" (at 355.6 199.9 0) (effects (font (size 1 1))))
+(property "Value" "U921 dVdT - LOW voltage sense" (at 355.6 202.9 0) (effects (font (size 1 1))))
+(property "Footprint" "TestPoint:TestPoint_Pad_1.5x1.5mm" (at 355.6 215.9 0) (effects (font (size 1 1)) (hide yes)))
+(pin "1")
+(instances (project "TripTracer_A23_Integration" (path "/a26d9b0c-7f10-4e5a-a65f-000000000064/a26d9b0c-7f10-4e5a-a65f-000000000065" (reference "TP949") (unit 1)))))
+(global_label "R6_DVDT" (shape bidirectional) (at 350.52 215.9 0) (effects (font (size 1 1)) (justify left)))
+(text "ROUND6 LAB ONLY: these pads are not in the original 23-position A23 project; inspect probe capacitance and differential pin limits at 58V. No unqualified PCB production." (at 20.32 285.75 0) (effects (font (size 1 1))))
+(embedded_fonts no)
+)
