File: hardware/kicad/TripTracer_A23_Integration/01_TPS26631_A23_INTEGRATED.kicad_sch (KiCad schematic)
At the start: 17 parts, among them Q941 SQM100N10-10_GE3 100V AEC, Q942 BSS138LT1G DRIVER PULLDOWN, U921 TPS26631PWPR

Commit message: TripPower A23 integration LAB: add real local 10k SHDN default-OFF pull-down and <=3.3V enable test point, separate from original 23-core; host AON/temp still OPEN
Parts:
- added R950: 10k 1pct SHDN_LOCAL_FAILSAFE_PULLDOWN, Resistor_SMD:R_1206_3216Metric, symbol Tripmaster_Sym:R
- added TP950: SHDN DEBUG <=3p3V, low OFF, not vehicle release, TestPoint:TestPoint_Pad_1.5x1.5mm, symbol TripPower_PGOOD:SignalPad
Connections:
- net GND: now also R950.2
- net A23_SHDN_SAFE_EN: now reaches U921.13 (SHDN)
- net A23_SHDN_SAFE_EN: now also R950.1, TP950.1 (PAD)
- no-connect marks 4 -> 3
Other:
- note added: "Integration clone ONLY: R950 10k locally pulls SHDN LOW by default (TI SHDN abs 5.5V), enable only with externally VALIDATED 0..3.3V HOST_RUN_SAFE. No automatic supply start until Host AON thermal/ACC interlock exists. Standalone A23 unchanged."
Changed lines of the file:
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@@
 (wire (pts (xy 279.4 147.32) (xy 284.48 147.32)) (stroke (width 0) (type default)))
 (global_label "ILIM_SET" (shape bidirectional) (at 284.48 147.32 0) (effects (font (size 1 1)) (justify left)))
-(no_connect (at 279.4 137.16))
 (wire (pts (xy 279.4 111.76) (xy 284.48 111.76)) (stroke (width 0) (type default)))
 (global_label "VIN_PROTECTED_UNFUSED" (shape bidirectional) (at 284.48 111.76 0) (effects (font (size 1 1)) (justify left)))
@@
 (global_label "R6_DVDT" (shape bidirectional) (at 350.52 215.9 0) (effects (font (size 1 1)) (justify left)))
 (text "ROUND6 LAB ONLY: these pads are not in the original 23-position A23 project; inspect probe capacitance and differential pin limits at 58V. No unqualified PCB production." (at 20.32 285.75 0) (effects (font (size 1 1))))
+(symbol (lib_id "Tripmaster_Sym:R") (at 323.85 228.6 0) (unit 1) (in_bom yes) (on_board yes) (dnp no)
+(property "Reference" "R950" (at 323.85 212.6 0) (effects (font (size 1 1))))
+(property "Value" "10k 1pct SHDN_LOCAL_FAILSAFE_PULLDOWN" (at 323.85 215.6 0) (effects (font (size 1 1))))
+(property "Footprint" "Resistor_SMD:R_1206_3216Metric" (at 323.85 228.6 0) (effects (font (size 1 1)) (hide yes)))
+(property "MPN" "AC1206FR-0710KL" (at 0 0 0) (effects (font (size 1 1)) (hide yes)))
+(pin "1")
+(pin "2")
+(instances (project "TripTracer_A23_Integration" (path "/a26d9b0c-7f10-4e5a-a65f-000000000064/a26d9b0c-7f10-4e5a-a65f-000000000065" (reference "R950") (unit 1)))))
+(global_label "A23_SHDN_SAFE_EN" (shape input) (at 279.4 137.16 0) (effects (font (size 1 1)) (justify left)))
+(global_label "A23_SHDN_SAFE_EN" (shape bidirectional) (at 312.42 228.6 0) (effects (font (size 1 1)) (justify left)))
+(global_label "GND" (shape bidirectional) (at 335.28 228.6 0) (effects (font (size 1 1)) (justify left)))
+(symbol (lib_id "TripPower_PGOOD:SignalPad") (at 355.6 228.6 0) (unit 1) (in_bom no) (on_board yes) (dnp no)
+(property "Reference" "TP950" (at 355.6 212.6 0) (effects (font (size 1 1))))
+(property "Value" "SHDN DEBUG <=3p3V, low OFF, not vehicle release" (at 355.6 215.6 0) (effects (font (size 1 1))))
+(property "Footprint" "TestPoint:TestPoint_Pad_1.5x1.5mm" (at 355.6 228.6 0) (effects (font (size 1 1)) (hide yes)))
+(pin "1")
+(instances (project "TripTracer_A23_Integration" (path "/a26d9b0c-7f10-4e5a-a65f-000000000064/a26d9b0c-7f10-4e5a-a65f-000000000065" (reference "TP950") (unit 1)))))
+(global_label "A23_SHDN_SAFE_EN" (shape bidirectional) (at 350.52 228.6 0) (effects (font (size 1 1)) (justify left)))
+(text "Integration clone ONLY: R950 10k locally pulls SHDN LOW by default (TI SHDN abs 5.5V), enable only with externally VALIDATED 0..3.3V HOST_RUN_SAFE. No automatic supply start until Host AON thermal/ACC interlock exists. Standalone A23 unchanged." (at 20.32 275.59 0) (effects (font (size 1 1))))
 (embedded_fonts no)
 )
